File: Small_Pendant/LEDs.kicad_sch (KiCad schematic)
At the start: 177 parts

Commit message: [HW] Make Pendant as separate module (no MCU)
Changed lines of the file:
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@@
 	)
 	(global_label "DATA_THRU5"
-		(shape input)
+		(shape output)
 		(at 146.05 195.58 180)
 		(fields_autoplaced yes)
@@
 	)
 	(global_label "DATA_THRU9"
-		(shape input)
+		(shape output)
 		(at 247.65 160.02 180)
 		(fields_autoplaced yes)
@@
 	)
 	(global_label "DATA_THRU8"
-		(shape input)
+		(shape output)
 		(at 222.25 160.02 180)
 		(fields_autoplaced yes)
@@
 	)
 	(global_label "DATA_THRU1"
-		(shape input)
+		(shape output)
 		(at 44.45 195.58 180)
 		(fields_autoplaced yes)
@@
 	)
 	(global_label "DATA_THRU7"
-		(shape input)
+		(shape output)
 		(at 196.85 160.02 180)
 		(fields_autoplaced yes)
@@
 	)
 	(global_label "DATA_THRU6"
-		(shape input)
+		(shape output)
 		(at 171.45 195.58 180)
 		(fields_autoplaced yes)
@@
 	)
 	(global_label "DATA_THRU3"
-		(shape input)
+		(shape output)
 		(at 95.25 195.58 180)
 		(fields_autoplaced yes)
@@
 	)
 	(global_label "DATA_THRU4"
-		(shape input)
+		(shape output)
 		(at 120.65 195.58 180)
 		(fields_autoplaced yes)
@@
 	)
 	(global_label "DATA_THRU2"
-		(shape input)
+		(shape output)
 		(at 69.85 195.58 180)
 		(fields_autoplaced yes)
