File: Small_Pendant/LEDs.kicad_sch (KiCad schematic)
At the start: 177 parts

Commit message: [HW] Add Buttons and Replace Transistors Picked a Connector, need to create symbol and footprint Need VREG, then that's all components Still lots of DRC issues
Parts:
- D1, D10, D100, D101, D102, D103, D104, D105, D106, D107, D108, D109, D11, D110, D111, D112, D113, D114, D115, D116, D117, D118, D119, D12, D120, D121, D122, D123, D124, D125, D126, D127, D128, D129, D13, D130, D131, D132, D133, D134, D135, D136, D137, D138, D139, D14, D140, D141, D142, D143, D144, D145, D146, D147, D148, D149, D15, D150, D151, D152, D153, D154, D155, D156, D157, D158, D159, D16, D160, D161, D162, D163, D164, D165, D166, D167, D168, D169, D17, D170, D171, D172, D173, D174, D175, D176, D177, D18, D19, D2, D20, D21, D22, D23, D24, D25, D26, D27, D28, D29, D3, D30, D31, D32, D33, D34, D35, D36, D37, D38, D39, D4, D40, D41, D42, D43, D44, D45, D46, D47, D48, D49, D5, D50, D51, D52, D53, D54, D55, D56, D57, D58, D59, D6, D60, D61, D62, D63, D64, D65, D66, D67, D68, D69, D7, D70, D71, D72, D73, D74, D75, D76, D77, D78, D79, D8, D80, D81, D82, D83, D84, D85, D86, D87, D88, D89, D9, D90, D91, D92, D93, D94, D95, D96, D97, D98, D99: Part# (none) -> C5349953

Commit message: [HW] Added ESD Diode, Added VREG TODO: Connectors TODO?: Status LEDs (PWR vs Boot) (LED built in is a good idea to have, could blink every second to show alive-ness)
Parts:
- renumbered D1 to D178
Changed lines of the file:
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@@
 		(on_board yes)
 		(dnp no)
-		(property "Reference" "D1"
+		(property "Reference" "D178"
 			(at 34.29 17.78 0)
 			(effects
@@
 			(project "Small_Pendant"
 				(path "/e1f67532-4244-48a0-a633-004c4e91cc2f/f7e054ab-e6f9-45d1-9e92-1309241566f0"
-					(reference "D1")
+					(reference "D178")
 					(unit 1)
 				)

Commit message: [HW] Re-annotate components, which absolutely wrecked everything, need to re-do the layout again
Parts:
- renumbered D8 to D10, D98 to D100, D99 to D101, D100 to D102, D101 to D103, D102 to D104, D103 to D105, D104 to D106, D105 to D107, D106 to D108, D107 to D109, D9 to D11, D108 to D110, D109 to D111, D110 to D112, D111 to D113, D112 to D114, D113 to D115, D114 to D116, D115 to D117, D116 to D118, D117 to D119, D10 to D12, D118 to D120, D119 to D121, D120 to D122, D121 to D123, D122 to D124, D123 to D125, D124 to D126, D125 to D127, D126 to D128, D127 to D129, D11 to D13, D128 to D130, D129 to D131, D130 to D132, D131 to D133, D132 to D134, D133 to D135, D134 to D136, D135 to D137, D136 to D138, D137 to D139, D12 to D14, D138 to D140, D139 to D141, D140 to D142, D141 to D143, D142 to D144, D143 to D145, D144 to D146, D145 to D147, D146 to D148, D147 to D149, D13 to D15, D148 to D150, D149 to D151, D150 to D152, D151 to D153, D152 to D154, D153 to D155, D154 to D156, D155 to D157, D156 to D158, D157 to D159, D14 to D16, D158 to D160, D159 to D161, D160 to D162, D161 to D163, D162 to D164, D163 to D165, D164 to D166, D165 to D167, D166 to D168, D167 to D169, D15 to D17, D168 to D170, D169 to D171, D170 to D172, D171 to D173, D172 to D174, D173 to D175, D174 to D176, D175 to D177, D176 to D178, D177 to D179, D16 to D18, D17 to D19, D18 to D20, D19 to D21, D20 to D22, D21 to D23, D22 to D24, D23 to D25, D24 to D26, D25 to D27, D26 to D28, D27 to D29, D178 to D3, D28 to D30, D29 to D31, D30 to D32, D31 to D33, D32 to D34, D33 to D35, D34 to D36, D35 to D37, D36 to D38, D37 to D39, D2 to D4, D38 to D40, D39 to D41, D40 to D42, D41 to D43, D42 to D44, D43 to D45, D44 to D46, D45 to D47, D46 to D48, D47 to D49, D3 to D5, D48 to D50, D49 to D51, D50 to D52, D51 to D53, D52 to D54, D53 to D55, D54 to D56, D55 to D57, D56 to D58, D57 to D59, D4 to D6, D58 to D60, D59 to D61, D60 to D62, D61 to D63, D62 to D64, D63 to D65, D64 to D66, D65 to D67, D66 to D68, D67 to D69, D5 to D7, D68 to D70, D69 to D71, D70 to D72, D71 to D73, D72 to D74, D73 to D75, D74 to D76, D75 to D77, D76 to D78, D77 to D79, D6 to D8, D78 to D80, D79 to D81, D80 to D82, D81 to D83, D82 to D84, D83 to D85, D84 to D86, D85 to D87, D86 to D88, D87 to D89, D7 to D9, D88 to D90, D89 to D91, D90 to D92, D91 to D93, D92 to D94, D93 to D95, D94 to D96, D95 to D97, D96 to D98, D97 to D99

Commit message: [HW] Added Connectors, P1.27mm double wide headers
Connections:
- net +5V renamed +5VL
- net Earth renamed GND

Commit message: [HW] switched J4/7 to 2x4 connectors for more current capacity
Parts:
- D10, D100, D101, D102, D103, D104, D105, D106, D107, D108, D109, D11, D110, D111, D112, D113, D114, D115, D116, D117, D118, D119, D12, D120, D121, D122, D123, D124, D125, D126, D127, D128, D129, D13, D130, D131, D132, D133, D134, D135, D136, D137, D138, D139, D14, D140, D141, D142, D143, D144, D145, D146, D147, D148, D149, D15, D150, D151, D152, D153, D154, D155, D156, D157, D158, D159, D16, D160, D161, D162, D163, D164, D165, D166, D167, D168, D169, D17, D170, D171, D172, D173, D174, D175, D176, D177, D178, D179, D18, D19, D20, D21, D22, D23, D24, D25, D26, D27, D28, D29, D3, D30, D31, D32, D33, D34, D35, D36, D37, D38, D39, D4, D40, D41, D42, D43, D44, D45, D46, D47, D48, D49, D5, D50, D51, D52, D53, D54, D55, D56, D57, D58, D59, D6, D60, D61, D62, D63, D64, D65, D66, D67, D68, D69, D7, D70, D71, D72, D73, D74, D75, D76, D77, D78, D79, D8, D80, D81, D82, D83, D84, D85, D86, D87, D88, D89, D9, D90, D91, D92, D93, D94, D95, D96, D97, D98, D99: LCSC Part (none) -> C5349953; Part# C5349953 -> (none)

Commit message: [HW] Add Series Resistor and power ESD diode
Parts:
- renumbered D9 to D10, D99 to D100, D100 to D101, D101 to D102, D102 to D103, D103 to D104, D104 to D105, D105 to D106, D106 to D107, D107 to D108, D108 to D109, D10 to D11, D109 to D110, D110 to D111, D111 to D112, D112 to D113, D113 to D114, D114 to D115, D115 to D116, D116 to D117, D117 to D118, D118 to D119, D11 to D12, D119 to D120, D120 to D121, D121 to D122, D122 to D123, D123 to D124, D124 to D125, D125 to D126, D126 to D127, D127 to D128, D128 to D129, D12 to D13, D129 to D130, D130 to D131, D131 to D132, D132 to D133, D133 to D134, D134 to D135, D135 to D136, D136 to D137, D137 to D138, D138 to D139, D13 to D14, D139 to D140, D140 to D141, D141 to D142, D142 to D143, D143 to D144, D144 to D145, D145 to D146, D146 to D147, D147 to D148, D148 to D149, D14 to D15, D149 to D150, D150 to D151, D151 to D152, D152 to D153, D153 to D154, D154 to D155, D155 to D156, D156 to D157, D157 to D158, D158 to D159, D15 to D16, D159 to D160, D160 to D161, D161 to D162, D162 to D163, D163 to D164, D164 to D165, D165 to D166, D166 to D167, D167 to D168, D168 to D169, D16 to D17, D169 to D170, D170 to D171, D171 to D172, D172 to D173, D173 to D174, D174 to D175, D175 to D176, D176 to D177, D177 to D178, D178 to D179, D17 to D18, D179 to D180, D18 to D19, D19 to D20, D20 to D21, D21 to D22, D22 to D23, D23 to D24, D24 to D25, D25 to D26, D26 to D27, D27 to D28, D28 to D29, D29 to D30, D30 to D31, D31 to D32, D32 to D33, D33 to D34, D34 to D35, D35 to D36, D36 to D37, D37 to D38, D38 to D39, D3 to D4, D39 to D40, D40 to D41, D41 to D42, D42 to D43, D43 to D44, D44 to D45, D45 to D46, D46 to D47, D47 to D48, D48 to D49, D4 to D5, D49 to D50, D50 to D51, D51 to D52, D52 to D53, D53 to D54, D54 to D55, D55 to D56, D56 to D57, D57 to D58, D58 to D59, D5 to D6, D59 to D60, D60 to D61, D61 to D62, D62 to D63, D63 to D64, D64 to D65, D65 to D66, D66 to D67, D67 to D68, D68 to D69, D6 to D7, D69 to D70, D70 to D71, D71 to D72, D72 to D73, D73 to D74, D74 to D75, D75 to D76, D76 to D77, D77 to D78, D78 to D79, D7 to D8, D79 to D80, D80 to D81, D81 to D82, D82 to D83, D83 to D84, D84 to D85, D85 to D86, D86 to D87, D87 to D88, D88 to D89, D8 to D9, D89 to D90, D90 to D91, D91 to D92, D92 to D93, D93 to D94, D94 to D95, D95 to D96, D96 to D97, D97 to D98, D98 to D99
