File: Small_Pendant/Small_Pendant.kicad_sch (KiCad schematic)
At the start: 0 parts

Commit message: [HW] Split Boards, need to move Caps for LEDs and add all the assorcted stuff for the ESP32
Changed lines of the file:
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@@
 		(comment 1 "Matthew Haahr")
 	)
-	(text_box "TODOs:\nESP32-C3 (or C6) Mini on Second board, can take advantage of WiFi\n\nhttps://docs.espressif.com/projects/esp-idf/en/v5.2/esp32c3/hw-reference/esp32c3/user-guide-devkitm-1.html\n\nFTDI FT234XD-R for USB-UART (setup AutoProg)\n\nOnly need a 3V3 Regulator and Level Shifter\n\nLSM6DSOX for IMU (use Libs for Abs Orientation)\n\nButtons:\n - Pattern Button (Scrolling Dot, Bouncing Dots, RGB, Fluid?)\n - Color Button (Color Cycle then Rainbow for solid color ones)\n - Sleep off the Pattern Button? (and wake from sleep)\n\nWiFi:\n - Basically the button interface (dropdown for pattern, color picker)\n\nPanelize on my own\n\nFigure out interboard connectors (want relatively high current)\n\nJust power over USB-C? (5V3A should be enough, needs testing with Power Supply)"
+	(text_box "TODOs:\nESP32-C3 (or C6) Mini on Second board, can take advantage of WiFi\n\nhttps://docs.espressif.com/projects/esp-idf/en/v5.2/esp32c3/hw-reference/esp32c3/user-guide-devkitm-1.html\n\nFTDI FT234XD-R for USB-UART (setup AutoProg)\n\nOnly need a 3V3 Regulator and Level Shifter\n\nLSM6DSOX for IMU (use Libs for Abs Orientation) (Or just BNO055, no code needed)\n\nButtons:\n - Pattern Button (Scrolling Dot, Bouncing Dots, RGB, Fluid?)\n - Color Button (Color Cycle then Rainbow for solid color ones)\n - Sleep off the Pattern Button? (and wake from sleep)\n\nWiFi:\n - Basically the button interface (dropdown for pattern, color picker)\n\nPanelize on my own\n\nFigure out interboard connectors (want relatively high current)\n\nJust power over USB-C? (5V3A should be enough, needs testing with Power Supply)\n\nStatus LEDs? (Power vs Boot (Make Disable-able?)"
 		(exclude_from_sim no)
 		(at 68.58 38.1 0)
-		(size 118.11 52.07)
+		(size 118.11 55.88)
 		(stroke
 			(width 0)

Commit message: [HW] Added IMU and corrected UART Bridge, all chip support components added, still need reset and boot connections though
Other:
- added sheet LED Support (LED-Support.kicad_sch)
Changed lines of the file:
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@@
 	)
 	(sheet
-		(at 17.78 46.99)
+		(at 17.78 48.26)
+		(size 31.75 20.32)
+		(fields_autoplaced yes)
+		(stroke
+			(width 0.1524)
+			(type solid)
+		)
+		(fill
+			(color 0 0 0 0.0000)
+		)
+		(property "Sheetname" "LED Support"
+			(at 17.78 47.5484 0)
+			(effects
+				(font
+					(size 1.27 1.27)
+				)
+				(justify left bottom)
+			)
+		)
+		(property "Sheetfile" "LED-Support.kicad_sch"
+			(at 17.78 69.1646 0)
+			(effects
+				(font
+					(size 1.27 1.27)
+				)
+				(justify left top)
+			)
+		)
+		(instances
+			(project "Small_Pendant"
+				(path "/e1f67532-4244-48a0-a633-004c4e91cc2f"
+					(page "4")
+				)
+			)
+		)
+	)
+	(sheet
+		(at 17.78 77.47)
 		(size 31.75 20.32)
 		(fields_autoplaced yes)
@@
 		)
 		(property "Sheetname" "MCU"
-			(at 17.78 46.2784 0)
+			(at 17.78 76.7584 0)
 			(effects
 				(font
@@
 		)
 		(property "Sheetfile" "MCU.kicad_sch"
-			(at 17.78 67.8946 0)
+			(at 17.78 98.3746 0)
 			(effects
 				(font

Commit message: [HW] Added ESD Diode, Added VREG TODO: Connectors TODO?: Status LEDs (PWR vs Boot) (LED built in is a good idea to have, could blink every second to show alive-ness)
Changed lines of the file:
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@@
 		(comment 1 "Matthew Haahr")
-	)
-	(text_box "TODOs:\nESP32-C3 (or C6) Mini on Second board, can take advantage of WiFi\n\nhttps://docs.espressif.com/projects/esp-idf/en/v5.2/esp32c3/hw-reference/esp32c3/user-guide-devkitm-1.html\n\nFTDI FT234XD-R for USB-UART (setup AutoProg)\n\nOnly need a 3V3 Regulator and Level Shifter\n\nLSM6DSOX for IMU (use Libs for Abs Orientation) (Or just BNO055, no code needed)\n\nButtons:\n - Pattern Button (Scrolling Dot, Bouncing Dots, RGB, Fluid?)\n - Color Button (Color Cycle then Rainbow for solid color ones)\n - Sleep off the Pattern Button? (and wake from sleep)\n\nWiFi:\n - Basically the button interface (dropdown for pattern, color picker)\n\nPanelize on my own\n\nFigure out interboard connectors (want relatively high current)\n\nJust power over USB-C? (5V3A should be enough, needs testing with Power Supply)\n\nStatus LEDs? (Power vs Boot (Make Disable-able?)"
-		(exclude_from_sim no)
-		(at 68.58 38.1 0)
-		(size 118.11 55.88)
-		(stroke
-			(width 0)
-			(type default)
-		)
-		(fill
-			(type none)
-		)
-		(effects
-			(font
-				(size 1.27 1.27)
-			)
-			(justify left top)
-		)
 	)
 	(sheet

Commit message: [HW] Schematic and Layout/Routing Clean Up
Other:
- note added: "All 177 RGB LEDs"
- note added: "Decoupling Caps Male Interboard Connectors"
- note added: "MCU USB Level Shift 3V3 Regulator Buttons Test Points Female Interboard Connectors"
Changed lines of the file:
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@@
 		(comment 1 "Matthew Haahr")
 	)
+	(text "All 177 RGB LEDs"
+		(exclude_from_sim no)
+		(at 19.05 47.244 0)
+		(effects
+			(font
+				(size 1.27 1.27)
+			)
+			(justify left top)
+		)
+	)
+	(text "Decoupling Caps\nMale Interboard Connectors"
+		(exclude_from_sim no)
+		(at 19.304 76.454 0)
+		(effects
+			(font
+				(size 1.27 1.27)
+			)
+			(justify left top)
+		)
+	)
+	(text "MCU\nUSB\nLevel Shift\n3V3 Regulator\nButtons\nTest Points\nFemale Interboard Connectors\n"
+		(exclude_from_sim no)
+		(at 18.796 19.304 0)
+		(effects
+			(font
+				(size 1.27 1.27)
+			)
+			(justify left top)
+		)
+	)
 	(sheet
-		(at 17.78 48.26)
+		(at 17.78 74.93)
 		(size 31.75 20.32)
 		(fields_autoplaced yes)
@@
 		)
 		(property "Sheetname" "LED Support"
-			(at 17.78 47.5484 0)
+			(at 17.78 74.2184 0)
 			(effects
 				(font
@@
 		)
 		(property "Sheetfile" "LED-Support.kicad_sch"
-			(at 17.78 69.1646 0)
+			(at 17.78 95.8346 0)
 			(effects
 				(font
@@
 	)
 	(sheet
-		(at 17.78 77.47)
+		(at 17.78 17.78)
 		(size 31.75 20.32)
 		(fields_autoplaced yes)
@@
 		)
 		(property "Sheetname" "MCU"
-			(at 17.78 76.7584 0)
+			(at 17.78 17.0684 0)
 			(effects
 				(font
@@
 		)
 		(property "Sheetfile" "MCU.kicad_sch"
-			(at 17.78 98.3746 0)
+			(at 17.78 38.6846 0)
+			(effects
+				(font
+					(size 1.27 1.27)
+				)
+				(justify left top)
+			)
+		)
+		(instances
+			(project "Small_Pendant"
+				(path "/e1f67532-4244-48a0-a633-004c4e91cc2f"
+					(page "2")
+				)
+			)
+		)
+	)
+	(sheet
+		(at 17.78 45.72)
+		(size 31.75 20.32)
+		(fields_autoplaced yes)
+		(stroke
+			(width 0.1524)
+			(type solid)
+		)
+		(fill
+			(color 0 0 0 0.0000)
+		)
+		(property "Sheetname" "LEDs"
+			(at 17.78 45.0084 0)
+			(effects
+				(font
+					(size 1.27 1.27)
+				)
+				(justify left bottom)
+			)
+		)
+		(property "Sheetfile" "LEDs.kicad_sch"
+			(at 17.78 66.6246 0)
 			(effects
 				(font
@@
 				)
 			)
-		)
-	)
-	(sheet
-		(at 17.78 19.05)
-		(size 31.75 20.32)
-		(fields_autoplaced yes)
-		(stroke
-			(width 0.1524)
-			(type solid)
-		)
-		(fill
-			(color 0 0 0 0.0000)
-		)
-		(property "Sheetname" "LEDs"
-			(at 17.78 18.3384 0)
-			(effects
-				(font
-					(size 1.27 1.27)
-				)
-				(justify left bottom)
-			)
-		)
-		(property "Sheetfile" "LEDs.kicad_sch"
-			(at 17.78 39.9546 0)
-			(effects
-				(font
-					(size 1.27 1.27)
-				)
-				(justify left top)
-			)
-		)
-		(instances
-			(project "Small_Pendant"
-				(path "/e1f67532-4244-48a0-a633-004c4e91cc2f"
-					(page "2")
-				)
-			)

Commit message: [Docs] Lots added to the Readme, BOM, schematics,...
Other:
- sheet LED Support renamed LED_Support
Changed lines of the file:
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@@
 			(color 0 0 0 0.0000)
 		)
-		(property "Sheetname" "LED Support"
+		(property "Sheetname" "LED_Support"
 			(at 17.78 74.2184 0)
 			(effects
