File: Small_Pendant/USB+Power.kicad_sch (KiCad schematic)
At the start: 11 parts, among them J1 USB_C_Receptacle_USB2.0_16P, U1 FT234XD-R

Commit message: [HW] Make 'lollipop' shaped for USB connector
Parts:
- J1: footprint Connector_USB:USB_C_Receptacle_GCT_USB4110 -> Connector_USB:USB_C_Receptacle_GCT_USB4105-xx-A_16P_TopMnt_Horizontal
Changed lines of the file:
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@@
 			)
 		)
-		(property "Footprint" "Connector_USB:USB_C_Receptacle_GCT_USB4110"
+		(property "Footprint" "Connector_USB:USB_C_Receptacle_GCT_USB4105-xx-A_16P_TopMnt_Horizontal"
 			(at 38.1 44.45 0)
 			(effects

Commit message: [HW] Update TODOs and combine USB Power Rails
Parts:
- removed C21, C22: 47pF, Capacitor_SMD:C_0402_1005Metric, symbol Device:C
- removed C23, C24: 100nF, Capacitor_SMD:C_0402_1005Metric, symbol Device:C
- removed C25: 4.7uF, Capacitor_SMD:C_0402_1005Metric, symbol Device:C
- removed C26: 10nF, Capacitor_SMD:C_0402_1005Metric, symbol Device:C
- removed J1: USB_C_Receptacle_USB2.0_16P, Connector_USB:USB_C_Receptacle_GCT_USB4105-xx-A_16P_TopMnt_Horizontal, symbol Connector:USB_C_Receptacle_USB2.0_16P
- removed R1: 0, Resistor_SMD:R_0402_1005Metric, symbol Device:R_US
- removed R2, R3: 27, Resistor_SMD:R_0402_1005Metric, symbol Device:R_US
- removed U1: FT234XD-R, Package_DFN_QFN:DFN-12-1EP_3x3mm_P0.45mm_EP1.65x2.38mm, symbol Interface_USB:FT234XD-R
Connections:
- no-connect marks 6 -> 0
