File: Small_Pendant/Capacitors.kicad_sch (KiCad schematic)
At the start: 20 parts

Commit message: [HW] Make Pendant as separate module (no MCU)
Parts:
- added J1: Conn_01x03, Connector_PinSocket_2.54mm:PinSocket_1x03_P2.54mm_Vertical_SMD_Pin1Right, symbol Connector_Generic:Conn_01x03
Connections:
- net +5V: now also J1.3 (Pin_3)
- net Earth: now also J1.1 (Pin_1)
- new net DATA_IN: J1.2 (Pin_2)

Commit message: [HW] Remove all microvias
Parts:
- J1: footprint Connector_PinSocket_2.54mm:PinSocket_1x03_P2.54mm_Vertical_SMD_Pin1Right -> Connector_PinHeader_2.54mm:PinHeader_1x03_P2.54mm_Horizontal
Changed lines of the file:
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@@
 			)
 		)
-		(property "Footprint" "Connector_PinSocket_2.54mm:PinSocket_1x03_P2.54mm_Vertical_SMD_Pin1Right"
+		(property "Footprint" "Connector_PinHeader_2.54mm:PinHeader_1x03_P2.54mm_Horizontal"
 			(at 27.94 100.33 0)
 			(effects
