File: Small_Pendant/Small_Pendant.kicad_pcb (KiCad board)
At the start: 4 copper layers, 28 x 28 mm, 205 parts, among them J1 USB_C_Receptacle_USB2.0_16P, U1 FT234XD-R, U2 SN74LVC1T45DCK

Commit message: [HW] Make 'lollipop' shaped for USB connector
Parts:
- J1: footprint Connector_USB:USB_C_Receptacle_GCT_USB4110 -> Connector_USB:USB_C_Receptacle_GCT_USB4105-xx-A_16P_TopMnt_Horizontal
- moved J1 4.25 mm to (50.0, 64.5)
- moved R1 4.25 mm to (54.0, 59.0)
- moved C24 1.89 mm to (42.3, 57.4)
- moved C25 1.89 mm to (42.3, 58.4)
- moved C26 1.89 mm to (43.8, 57.8)
- moved C23 1.66 mm to (43.1, 52.1)
- moved R2 1.66 mm to (45.8, 55.2)
- moved R3 1.66 mm to (45.8, 54.2)
- moved U1 1.66 mm to (42.9, 54.7)
- moved C21 1.66 mm to (47.8, 55.7)
- moved C22 1.66 mm to (47.8, 53.7)
Routing:
- net +3V3_USB: track 9.19 -> 6.01 mm
- net USB_D+: track 9.87 -> 12.5 mm
- net USB_D-: track 9.28 -> 11.9 mm
- net VUSB: track 14.8 -> 16.2 mm
- net Earth: track 23.8 -> 23.1 mm, vias 30 -> 27
- net Net-(J1-SHIELD): track 19.9 -> 19.5 mm, vias 2 -> 0
- net +5V: vias 21 -> 22
Other:
- board size 28 x 28 mm -> 24.9 x 30.7 mm

Commit message: [HW] Re-arrange and clean up, all current components placed
Parts:
- moved C22 5.24 mm to (51.0, 57.9), turned to 0 degrees
- moved R3 5.03 mm to (50.5, 55.9), turned to 90 degrees
- moved R2 3.81 mm to (49.5, 55.9), turned to 90 degrees
- moved C21 2.51 mm to (49.0, 57.9), turned to 180 degrees
- moved C23 1.99 mm to (45.1, 51.8)
- moved U1 1.99 mm to (44.9, 54.5)
- moved C24 0.99 mm to (43.3, 57.1)
- moved C25 0.99 mm to (43.3, 58.1)
- moved C26 0.99 mm to (44.7, 57.5)
Routing:
- net USB_D+: track 12.5 -> 7.31 mm
- net /USB+Power/USB_D'+: track 1.60 -> 6.55 mm
- net /USB+Power/USB_D'-: track 1.60 -> 6.52 mm
- net USB_D-: track 11.9 -> 7.31 mm
- net VUSB: track 16.2 -> 15.7 mm
- net Earth: track 23.1 -> 23.3 mm, vias 27 -> 28

Commit message: [HW] Update TODOs and combine USB Power Rails
Parts:
- removed C23, C24: 100nF, Capacitor_SMD:C_0402_1005Metric
- removed C25: 4.7uF, Capacitor_SMD:C_0402_1005Metric
- removed C26: 10nF, Capacitor_SMD:C_0402_1005Metric
- added C15: 100nF, Capacitor_SMD:C_0402_1005Metric, B.Cu at (44.6, 51.3)
- added C16: 100nF, Capacitor_SMD:C_0402_1005Metric, B.Cu at (44.7, 57.5)
- added C19: 4.7uF, Capacitor_SMD:C_0402_1005Metric, B.Cu at (43.3, 57.1)
- added C20: 10nF, Capacitor_SMD:C_0402_1005Metric, B.Cu at (43.3, 58.1)
Connections:
- net /USB+Power/USB_D'+ renamed /MCU/USB_D'+
- net /USB+Power/USB_D'- renamed /MCU/USB_D'-
- U1 pad 2: +3V3_USB -> +3V3
- U1 pad 3: +3V3_USB -> +3V3
- U1 pad 6: ON_CHARGE -> unconnected-(U1-CBUS0-Pad6)
- U1 pad 9: +3V3_USB -> +3V3
Routing:
- net +3V3: track 1.32 -> 18.4 mm, vias 0 -> 3
- net +3V3_USB: track 6.44 -> 0.00 mm, vias 2 -> 0
- net Earth: track 23.3 -> 23.4 mm, vias 28 -> 27

Commit message: [HW] Remove Blind Vias, add 5k1 CC resistors for 5V3A USB-C TODO: 3V3 Regulator (May switch FTDI to that) TODO: MCU (OSC?)
Parts:
- added C23: 1uF, Capacitor_SMD:C_0402_1005Metric, B.Cu at (46.8, 60.5)
- added C24: 10uF, Capacitor_SMD:C_0402_1005Metric, B.Cu at (53.2, 60.5)
- added G***: LOGO, Graphics:Logo, F.Cu at (50.0, 65.9)
- added R4: 5k1, Resistor_SMD:R_0402_1005Metric, B.Cu at (48.2, 60.0)
- added R5: 5k1, Resistor_SMD:R_0402_1005Metric, B.Cu at (51.8, 60.0)
- moved R1 1.73 mm to (55.2, 60.2)
- moved J1 1.32 mm to (50.0, 65.9)
- moved R2 0.86 mm to (49.5, 55.0)
- moved R3 0.86 mm to (50.5, 55.0)
- moved C18 0.82 mm to (49.1, 43.4)
- moved U2 0.82 mm to (51.1, 42.9)
- moved C17 0.72 mm to (50.8, 40.8)
- turned C15 to -90 degrees
- turned C16 to 90 degrees
Connections:
- C15 pad 1: +3V3 -> Earth
- C15 pad 2: Earth -> +3V3
- C16 pad 1: VUSB -> Earth
- C16 pad 2: Earth -> +5V
- C19 pad 1: VUSB -> +5V
- C20 pad 1: VUSB -> +5V
- J1 pad A4: VUSB -> +5V
- J1 pad A5: unconnected-(J1-CC1-PadA5) -> Net-(J1-CC1)
- J1 pad A9: VUSB -> +5V
- J1 pad B4: VUSB -> +5V
- J1 pad B5: unconnected-(J1-CC2-PadB5) -> Net-(J1-CC2)
- J1 pad B9: VUSB -> +5V
- U1 pad 4: VUSB -> +5V
Routing:
- net VUSB: track 15.7 -> 0.00 mm, vias 3 -> 0
- net +3V3: track 18.4 -> 3.02 mm, vias 3 -> 0
- net Earth: track 23.4 -> 38.2 mm, vias 27 -> 29
- net +5V: track 14.6 -> 21.9 mm, vias 22 -> 21
- net DATA_IN: track 2.21 -> 5.29 mm, vias 2 -> 1
- net USB_D-: track 7.31 -> 9.49 mm
- net USB_D+: track 7.31 -> 9.49 mm
- net Net-(J1-CC1): track 0.00 -> 1.88 mm
- net Net-(J1-CC2): track 0.00 -> 1.68 mm
- net /MCU/USB_D'-: track 6.52 -> 7.51 mm
- net /MCU/USB_D'+: track 6.55 -> 7.55 mm
- net Net-(J1-SHIELD): track 19.5 -> 20.4 mm
- removed copper zone on B.Cu, net VUSB
Other:
- board size 24.9 x 30.7 mm -> 24.9 x 32 mm

Commit message: [HW] Split Boards, need to move Caps for LEDs and add all the assorcted stuff for the ESP32
Parts:
- added U3: ESP32-C3-MINI-1, MCU_Espressif_Official:ESP32-C3-MINI-1, F.Cu at (95.4, 57.6)
- J1: moved to F.Cu
- moved G*** 46.2 mm to (48.2, 112.0)
- moved C10 41.1 mm to (57.9, 87.9)
- moved C18 41.1 mm to (46.5, 84.4)
- moved U2 41.1 mm to (48.5, 83.9)
- moved C1 41.1 mm to (44.4, 80.5)
- moved C11 41.1 mm to (56.4, 85.0)
- moved C12 41.1 mm to (54.9, 83.5)
- moved C13 41.1 mm to (53.4, 82.0)
- moved C14 41.1 mm to (50.4, 80.5)
- moved C16 41.1 mm to (42.1, 98.5)
- moved C17 41.1 mm to (48.1, 81.8)
- moved C2 41.1 mm to (41.4, 82.0)
- moved C23 41.1 mm to (44.1, 101.5)
- moved C24 41.1 mm to (50.6, 101.5)
- moved C3 41.1 mm to (39.9, 83.5)
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Routing:
- net Earth: track 38.2 -> 0.00 mm, vias 29 -> 14
- net +5V: track 21.9 -> 0.78 mm, vias 21 -> 14
- net Net-(J1-SHIELD): track 20.4 -> 0.00 mm
- net USB_D+: track 9.49 -> 0.00 mm
- net /MCU/USB_D'+: track 7.55 -> 0.00 mm
- net /MCU/USB_D'-: track 7.51 -> 0.00 mm
- net USB_D-: track 9.49 -> 2.38 mm, vias 2 -> 0
- net DATA_IN: track 5.29 -> 1.29 mm, vias 1 -> 0
- net +3V3: track 3.02 -> 0.00 mm
- net Net-(J1-CC1): track 1.88 -> 0.00 mm
- net Net-(J1-CC2): track 1.68 -> 0.00 mm
- net Net-(D66-DO): track 1.87 -> 2.50 mm
- removed copper zone on B.Cu, net +5V
- removed copper zone on B.Cu, net Earth
Other:
- board size 24.9 x 32 mm -> 55 x 25 mm

Commit message: [HW] Figure out MCU board shape and add power and ground planes
Parts:
- G***, U3: moved to B.Cu
- moved G*** 62.0 mm to (50.0, 50.0), turned to 180 degrees
- moved C17 38.5 mm to (81.1, 101.7)
- moved C18 38.5 mm to (79.5, 104.4)
- moved U2 38.5 mm to (81.5, 103.9)
- moved C22 27.0 mm to (70.3, 114.7)
- moved C21 27.0 mm to (68.3, 114.7)
- moved C23 27.0 mm to (66.1, 117.3)
- moved C24 27.0 mm to (72.5, 117.3)
- moved R1 27.0 mm to (74.5, 117.0)
- moved R2 27.0 mm to (68.8, 111.8)
- moved R3 27.0 mm to (69.8, 111.8)
- moved R4 27.0 mm to (67.5, 116.8)
- moved R5 27.0 mm to (71.0, 116.8)
- moved U3 17.9 mm to (80.2, 48.3), turned to 180 degrees
- moved C16 11.5 mm to (32.9, 105.4)
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Connections:
- U1 pad 10: EXT_RX -> EXT_TX
- U1 pad 7: EXT_TX -> EXT_RX
- U3 pad 1: Net-(U3-GND-Pad1) -> Earth
- U3 pad 11: Net-(U3-GND-Pad1) -> Earth
- U3 pad 14: Net-(U3-GND-Pad1) -> Earth
- U3 pad 2: Net-(U3-GND-Pad1) -> Earth
- U3 pad 3: unconnected-(U3-3V3-Pad3) -> +3V3
- U3 pad 30: unconnected-(U3-GPIO20/U0RXD-Pad30) -> EXT_RX
- U3 pad 31: unconnected-(U3-GPIO21/U0TXD-Pad31) -> EXT_TX
- U3 pad 36: Net-(U3-GND-Pad1) -> Earth
- U3 pad 37: Net-(U3-GND-Pad1) -> Earth
- U3 pad 38: Net-(U3-GND-Pad1) -> Earth
- U3 pad 39: Net-(U3-GND-Pad1) -> Earth
- U3 pad 40: Net-(U3-GND-Pad1) -> Earth
- U3 pad 41: Net-(U3-GND-Pad1) -> Earth
- U3 pad 42: Net-(U3-GND-Pad1) -> Earth
- U3 pad 43: Net-(U3-GND-Pad1) -> Earth
- U3 pad 44: Net-(U3-GND-Pad1) -> Earth
- U3 pad 45: Net-(U3-GND-Pad1) -> Earth
- U3 pad 46: Net-(U3-GND-Pad1) -> Earth
- U3 pad 47: Net-(U3-GND-Pad1) -> Earth
- U3 pad 48: Net-(U3-GND-Pad1) -> Earth
- U3 pad 49: Net-(U3-GND-Pad1) -> Earth
- U3 pad 50: Net-(U3-GND-Pad1) -> Earth
- U3 pad 51: Net-(U3-GND-Pad1) -> Earth
- U3 pad 52: Net-(U3-GND-Pad1) -> Earth
- U3 pad 53: Net-(U3-GND-Pad1) -> Earth
Routing:
- net Earth: track 0.00 -> 23.7 mm, vias 14 -> 34
- net USB_D-: track 2.38 -> 0.00 mm
- net +5V: vias 14 -> 20
- added copper zone on B.Cu, net Earth
Other:
- board size 55 x 25 mm -> 55 x 27.8 mm

Commit message: [HW] Added IMU and corrected UART Bridge, all chip support components added, still need reset and boot connections though
Parts:
- removed R1: 0, Resistor_SMD:R_0402_1005Metric
- added C25: 10uF, Capacitor_SMD:C_0402_1005Metric, F.Cu at (96.4, 60.5)
- added C26: 100nF, Capacitor_SMD:C_0402_1005Metric, F.Cu at (96.4, 62.5)
- added C27: 1uF, Capacitor_SMD:C_0402_1005Metric, F.Cu at (92.4, 63.3)
- added C28: 1uf, Capacitor_SMD:C_0402_1005Metric, F.Cu at (71.9, 54.9)
- added C29: 120nF, Capacitor_SMD:C_0402_1005Metric, F.Cu at (78.2, 46.9)
- added G***: LOGO, Graphics:Logo, F.Cu at (80.0, 41.2)
- added R10: 1k, Resistor_SMD:R_0402_1005Metric, F.Cu at (71.0, 46.4)
- added R11: 22k, Resistor_SMD:R_0402_1005Metric, F.Cu at (71.9, 56.9)
- added R12: 47k, Resistor_SMD:R_0402_1005Metric, F.Cu at (71.9, 55.9)
- added R13: 10k, Resistor_SMD:R_0402_1005Metric, F.Cu at (101.6, 49.3)
- added R14: 10k, Resistor_SMD:R_0402_1005Metric, F.Cu at (98.3, 49.4)
- added R6: 10k, Resistor_SMD:R_0402_1005Metric, F.Cu at (92.4, 59.9)
- added R7: 3.3k, Resistor_SMD:R_0402_1005Metric, F.Cu at (87.8, 50.1)
- added R8: 3.3k, Resistor_SMD:R_0402_1005Metric, F.Cu at (87.8, 51.1)
- added R9: 10k, Resistor_SMD:R_0402_1005Metric, B.Cu at (69.3, 49.8)
- added U4: BNO055, BNO055:LGA28R50P4X10_380X520X100, F.Cu at (80.0, 50.0)
- C15, C21, C22, R2, R3, R4, R5: moved to F.Cu
- C16: value 100nF -> 10uF; moved to F.Cu
- C19: value 4.7uF -> 1uF; moved to F.Cu
- C20: value 10nF -> 100nF; moved to F.Cu
- U1: value FT234XD-R -> CP2102N-Axx-xQFN24; footprint Package_DFN_QFN:DFN-12-1EP_3x3mm_P0.45mm_EP1.65x2.38mm -> Package_DFN_QFN:QFN-24-1EP_4x4mm_P0.5mm_EP2.6x2.6mm; moved to F.Cu
- moved C20 72.9 mm to (76.5, 48.6), turned to -90 degrees
- moved C19 71.1 mm to (79.7, 52.8), turned to 0 degrees
- moved C16 70.8 mm to (72.0, 46.4)
- moved C15 66.1 mm to (73.0, 46.4)
- moved C17 64.7 mm to (92.9, 38.1)
- moved C18 64.7 mm to (91.3, 40.8)
- moved U2 64.7 mm to (93.3, 40.3)
- moved U1 64.5 mm to (70.7, 50.0), turned to 180 degrees
- moved R4 62.6 mm to (82.9, 56.1), turned to 0 degrees
- moved R2 62.6 mm to (74.4, 49.5), turned to 180 degrees
- moved R3 61.5 mm to (74.4, 50.5), turned to 180 degrees
- moved R5 61.0 mm to (77.1, 56.1), turned to 0 degrees
- moved C21 59.9 mm to (81.0, 56.1), turned to 0 degrees
- moved C22 59.2 mm to (79.0, 56.1), turned to 180 degrees
- moved C23 54.6 mm to (69.3, 62.8)
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Connections:
- C16 pad 1: Earth -> +3V3
- C16 pad 2: +5V -> Earth
- C19 pad 1: +5V -> Net-(U4-CAP)
- C20 pad 1: +5V -> Earth
- C20 pad 2: Earth -> +3V3
- J1 pad S1: Net-(J1-SHIELD) -> unconnected-(J1-SHIELD-PadS1)_2
- U1 pad 1: /MCU/USB_D'- -> unconnected-(U1-~{RI}/CLK-Pad1)
- U1 pad 10: EXT_TX -> unconnected-(U1-NC-Pad10)
- U1 pad 12: /MCU/USB_D'+ -> unconnected-(U1-RS485/GPIO.2-Pad12)
- U1 pad 13: Earth -> unconnected-(U1-~{RXT}/GPIO.1-Pad13)
- U1 pad 2: +3V3 -> Earth
- U1 pad 3: +3V3 -> /MCU/USB_D'+
- U1 pad 4: +5V -> /MCU/USB_D'-
- U1 pad 5: Earth -> +3V3
- U1 pad 6: unconnected-(U1-CBUS0-Pad6) -> +3V3
- U1 pad 7: EXT_RX -> +3V3
- U1 pad 8: unconnected-(U1-RTS#-Pad8) -> VBUS_DET
- U1 pad 9: +3V3 -> Net-(U1-~{RST})
- U2 pad 3: DATA_IN -> LED_DATA-5V
- U3 pad 19: unconnected-(U3-GPIO5/ADC2_CH0-Pad19) -> IMU_INT
- U3 pad 23: unconnected-(U3-GPIO9-Pad23) -> GPIO9/BOOT
- U3 pad 5: unconnected-(U3-GPIO2/ADC1_CH2-Pad5) -> SDA
- U3 pad 6: unconnected-(U3-GPIO3/ADC1_CH3-Pad6) -> SCL
- U3 pad 8: unconnected-(U3-EN/CHIP_PU-Pad8) -> CHIP_EN
Routing:
- net VBUS_DET: track 0.00 -> 16.5 mm, vias 0 -> 2
- net Earth: track 23.7 -> 37.2 mm, vias 34 -> 44
- net USB_D-: track 0.00 -> 12.8 mm
- net USB_D+: track 0.00 -> 12.8 mm
- net +5V: track 0.78 -> 11.5 mm, vias 20 -> 21
- net IMU_INT: track 0.00 -> 9.02 mm, vias 0 -> 1
- net EXT_TX: track 0.00 -> 7.23 mm, vias 0 -> 1
- net SDA: track 0.00 -> 5.95 mm, vias 0 -> 1
- net EXT_RX: track 0.00 -> 5.89 mm, vias 0 -> 1
- net SCL: track 0.00 -> 5.74 mm, vias 0 -> 1
- net Net-(J1-CC1): track 0.00 -> 5.45 mm
- net +3V3: track 0.00 -> 3.14 mm, vias 0 -> 7
- net Net-(J1-CC2): track 0.00 -> 2.08 mm
- net Net-(U1-~{SUSPEND}): track 0.00 -> 1.72 mm, vias 0 -> 1
- net /MCU/USB_D'-: track 0.00 -> 1.41 mm
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- added copper zone on F.Cu, net +3V3
- added copper zone on In1.Cu, net +3V3

Commit message: [HW] Move Support Components in
Parts:
- C25, C26, C27, R6: moved to B.Cu
- moved C18 22.4 mm to (69.9, 47.4), turned to -90 degrees
- moved C17 22.1 mm to (71.5, 43.7)
- moved U2 22.1 mm to (71.9, 45.9)
- moved R13 18.2 mm to (84.2, 54.8)
- moved C26 17.0 mm to (89.2, 47.1), turned to 180 degrees
- moved C25 16.1 mm to (89.2, 46.1), turned to 180 degrees
- moved R14 14.6 mm to (83.8, 48.4), turned to -90 degrees
- moved C23 14.3 mm to (82.8, 57.9), turned to 0 degrees
- moved C27 8.06 mm to (89.7, 55.7), turned to -90 degrees
- moved C24 6.67 mm to (77.2, 57.9), turned to 180 degrees
- moved R6 5.60 mm to (88.7, 55.7), turned to 90 degrees
Connections:
- U3 pad 22: unconnected-(U3-GPIO8-Pad22) -> LED_DATA
Routing:
- net LED_DATA: track 0.00 -> 12.5 mm
- net Earth: track 37.2 -> 45.2 mm, vias 44 -> 49
- net Net-(U4-NBOOT_LOAD_PIN): track 0.00 -> 7.04 mm
- net CHIP_EN: track 0.00 -> 5.73 mm
- net Net-(U4-NRESET): track 0.00 -> 5.65 mm
- net DATA_IN: track 1.29 -> 0.00 mm, vias 0 -> 1
- net +5V: track 11.5 -> 12.8 mm, vias 21 -> 22
- net +3V3: track 3.14 -> 4.24 mm, vias 7 -> 12
- net SDA: track 5.95 -> 6.48 mm
