File: Small_Pendant/Small_Pendant.kicad_pcb (KiCad board)
At the start: 4 copper layers, 56.6 x 27.6 mm, 232 parts, among them J1 USB_C_Receptacle_USB2.0_16P, J2 Interboard, J3 Interboard, J4 Interboard, J5 Interboard, J6 Interboard, J7 Interboard, SW1 SW_Push, SW2 SW_Push, SW3 SW_Push, U1 ESP32-C3-MINI-1, U2 AP2112K-3.3, U3 BNO055, U4 SN74LVC1T45DCK

Commit message: [HW] Add LED (green) That's all the parts, now need to spec caps and resistors
Parts:
- added D2: BLUE, LED_SMD:LED_0603_1608Metric, F.Cu at (87.8, 57.3)
- added R4: 1k3, Resistor_SMD:R_0402_1005Metric, F.Cu at (86.1, 57.6)
Routing:
- net /MCU/LED_BUILTIN: track 0.00 -> 4.66 mm, vias 0 -> 1
- net Net-(D2-A): track 0.00 -> 1.70 mm
- net DATA_IN: track 13.0 -> 11.9 mm
- net Earth: track 54.1 -> 53.2 mm, vias 21 -> 22
- net +5VL: track 37.3 -> 36.5 mm
- net Net-(J2-Pin_3): track 4.45 -> 3.85 mm
- net +5V: track 54.0 -> 53.5 mm

Commit message: [HW] Add Test Points [SW] Update the board configs correctly
Parts:
- added TP1: TX, TestPoint:TestPoint_Pad_0.5x0.5mm, B.Cu at (67.9, 49.5)
- added TP2: RX, TestPoint:TestPoint_Pad_0.5x0.5mm, B.Cu at (67.9, 50.4)
- added TP3: 3V3, TestPoint:TestPoint_Pad_0.5x0.5mm, B.Cu at (90.1, 56.9)
- added TP4: 5V, TestPoint:TestPoint_Pad_0.5x0.5mm, B.Cu at (91.1, 55.5)
- added TP5: GND, TestPoint:TestPoint_Pad_0.5x0.5mm, B.Cu at (89.1, 58.3)
Connections:
- U1 pad 30: unconnected-(U1-GPIO20/U0RXD-Pad30) -> Net-(U1-GPIO20/U0RXD)
- U1 pad 31: unconnected-(U1-GPIO21/U0TXD-Pad31) -> Net-(U1-GPIO21/U0TXD)
Routing:
- net Net-(U1-GPIO20/U0RXD): track 0.00 -> 6.61 mm
- net Net-(U1-GPIO21/U0TXD): track 0.00 -> 6.32 mm
- net Earth: track 53.2 -> 58.8 mm
- net +5V: track 53.5 -> 57.8 mm
- net +3V3: track 10.00 -> 12.6 mm, vias 7 -> 8
- net USR_BTN: track 7.23 -> 9.06 mm
- net GPIO9/BOOT: track 12.2 -> 10.5 mm

Commit message: [HW] switched J4/7 to 2x4 connectors for more current capacity
Parts:
- D2: value BLUE -> GREEN
- J4: footprint Connector_PinSocket_1.27mm:PinSocket_2x02_P1.27mm_Vertical_SMD -> Connector_PinSocket_1.27mm:PinSocket_2x04_P1.27mm_Vertical_SMD
- J7: footprint Connector_PinHeader_1.27mm:PinHeader_2x02_P1.27mm_Vertical_SMD -> Connector_PinHeader_1.27mm:PinHeader_2x04_P1.27mm_Vertical_SMD
- moved J4 0.20 mm to (89.9, 50.0)
- moved J7 0.20 mm to (40.1, 50.0)
Connections:
- J4 pad 3: Earth -> +5V
- J4 pad 4: Earth -> +5V
- J7 pad 3: GND -> +5VL
- J7 pad 4: GND -> +5VL
Routing:
- net Earth: track 58.8 -> 70.6 mm
- net +5V: track 57.8 -> 63.5 mm
- net +5VL: track 36.5 -> 40.2 mm
- net GND: track 34.9 -> 37.7 mm

Commit message: [HW] Schematic and Layout/Routing Clean Up
Parts:
- moved C28 1.50 mm to (51.5, 39.5)
- turned R4 to 90 degrees
Connections:
- net Net-(J2-Pin_3) renamed LED_DATA_5V
- R4 pad 1: /MCU/LED_BUILTIN -> Net-(D2-A)
- R4 pad 2: Net-(D2-A) -> /MCU/LED_BUILTIN
Routing:
- net +5VL: track 40.2 -> 25.5 mm, vias 14 -> 20
- net GND: track 37.7 -> 27.7 mm, vias 14 -> 21

Commit message: [HW] Clean up ESD Diode
Parts:
- moved D1 6.92 mm to (79.5, 54.1), turned to -90 degrees
- moved C12 2.00 mm to (80.2, 52.7), turned to 0 degrees
- moved R11 0.51 mm to (77.6, 55.4)
Connections:
- D1 pad 1: /MCU/USB_D'- -> USB_D+
- D1 pad 2: /MCU/USB_D'+ -> USB_D-
Routing:
- net Earth: track 70.6 -> 75.1 mm, vias 22 -> 21
- net /MCU/USB_D'+: track 2.18 -> 1.18 mm
- net /MCU/USB_D'-: track 2.18 -> 1.18 mm
- net Net-(J1-CC1): track 2.45 -> 1.89 mm
- net USB_D-: track 9.37 -> 9.93 mm
- net USB_D+: track 9.43 -> 9.96 mm
