File: Small_Pendant/Small_Pendant.kicad_pcb (KiCad board)
At the start: 4 copper layers, 56.6 x 27.6 mm, 239 parts, among them J1 USB_C_Receptacle_USB2.0_16P, J2 Interboard, J3 Interboard, J4 Interboard, J5 Interboard, J6 Interboard, J7 Interboard, SW1 SW_Push, SW2 SW_Push, SW3 SW_Push, U1 ESP32-C3-MINI-1, U2 AP2112K-3.3, U3 BNO055, U4 SN74LVC1T45DCK

Commit message: [HW] Add Series Resistor and power ESD diode
Parts:
- removed the D3 at (52.9, 39.5)
- added D180: XL-1010RGBC-WS2812B, LED_SMD:XINGLIGHT-XL-1010RGBC, F.Cu at (47.0, 60.5)
- added D2: ESD441DPLR, EasyEDA2KiCad:X2SON-2_L0.6-W0.3-P0.35_ESD441DPLR, B.Cu at (81.6, 58.1)
- added R12: 470, Resistor_SMD:R_0402_1005Metric, B.Cu at (56.0, 42.5)
- moved D175 3.35 mm to (56.0, 59.0), turned to 180 degrees
- moved D8 3.35 mm to (47.0, 39.5), turned to 0 degrees
- moved D17 2.19 mm to (56.0, 41.0), turned to 180 degrees
- moved D129 2.12 mm to (60.5, 53.0), turned to 180 degrees
- moved D155 2.12 mm to (59.0, 56.0), turned to 180 degrees
- moved D166 2.12 mm to (42.5, 57.5), turned to 0 degrees
- moved D28 2.12 mm to (42.5, 42.5), turned to 0 degrees
- moved D54 2.12 mm to (41.0, 45.5), turned to 0 degrees
- moved D4 1.60 mm to (53.0, 39.5)
- moved D5 1.60 mm to (51.5, 39.5)
- moved D10 1.50 mm to (45.5, 41.0)
- moved D100 1.50 mm to (60.5, 51.5)
- moved D101 1.50 mm to (59.0, 51.5)
- moved D102 1.50 mm to (57.5, 51.5)
- moved D103 1.50 mm to (56.0, 51.5)
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- renumbered D2 to D3
Connections:
- D102 pad 1: DATA_THRU5 -> Net-(D102-DO)
- D103 pad 1: Net-(D103-DO) -> DATA_THRU5
- D103 pad 4: DATA_THRU5 -> Net-(D102-DO)
- D104 pad 4: Net-(D103-DO) -> DATA_THRU5
- D122 pad 1: DATA_THRU6 -> Net-(D122-DO)
- D123 pad 1: Net-(D123-DO) -> DATA_THRU6
- D123 pad 4: DATA_THRU6 -> Net-(D122-DO)
- D124 pad 4: Net-(D123-DO) -> DATA_THRU6
- D138 pad 1: DATA_THRU7 -> Net-(D138-DO)
- D139 pad 1: Net-(D139-DO) -> DATA_THRU7
- D139 pad 4: DATA_THRU7 -> Net-(D138-DO)
- D140 pad 4: Net-(D139-DO) -> DATA_THRU7
- D154 pad 1: DATA_THRU8 -> Net-(D154-DO)
- D155 pad 1: Net-(D155-DO) -> DATA_THRU8
- D155 pad 4: DATA_THRU8 -> Net-(D154-DO)
- D156 pad 4: Net-(D155-DO) -> DATA_THRU8
- D170 pad 1: DATA_THRU9 -> Net-(D170-DO)
- D171 pad 1: Net-(D171-DO) -> DATA_THRU9
- D171 pad 4: DATA_THRU9 -> Net-(D170-DO)
- D172 pad 4: Net-(D171-DO) -> DATA_THRU9
- D179 pad 1: unconnected-(D179-DO-Pad1) -> Net-(D179-DO)
- D22 pad 1: DATA_THRU1 -> Net-(D22-DO)
- D23 pad 1: Net-(D23-DO) -> DATA_THRU1
- D23 pad 4: DATA_THRU1 -> Net-(D22-DO)
- D24 pad 4: Net-(D23-DO) -> DATA_THRU1
- D4 pad 4: Net-(D3-DO) -> DATA_IN
- D42 pad 1: DATA_THRU2 -> Net-(D42-DO)
- D43 pad 1: Net-(D43-DO) -> DATA_THRU2
- D43 pad 4: DATA_THRU2 -> Net-(D42-DO)
- D44 pad 4: Net-(D43-DO) -> DATA_THRU2
- D62 pad 1: DATA_THRU3 -> Net-(D62-DO)
- D63 pad 1: Net-(D63-DO) -> DATA_THRU3
- D63 pad 4: DATA_THRU3 -> Net-(D62-DO)
- D64 pad 4: Net-(D63-DO) -> DATA_THRU3
- D82 pad 1: DATA_THRU4 -> Net-(D82-DO)
- D83 pad 1: Net-(D83-DO) -> DATA_THRU4
- D83 pad 4: DATA_THRU4 -> Net-(D82-DO)
- D84 pad 4: Net-(D83-DO) -> DATA_THRU4
- J5 pad 3: DATA_IN -> Net-(J5-Pin_3)
- J5 pad 4: DATA_IN -> Net-(J5-Pin_3)
Routing:
- net Net-(J5-Pin_3): track 0.00 -> 9.47 mm
- net DATA_IN: track 11.8 -> 3.93 mm
- net Net-(D16-DO): track 3.97 -> 0.92 mm
- net Net-(D17-DO): track 0.92 -> 3.97 mm
- net Net-(D8-DO): track 0.92 -> 3.86 mm
- net Net-(D7-DO): track 3.86 -> 0.92 mm
- net Net-(D175-DO): track 0.92 -> 3.81 mm
- net Net-(D174-DO): track 3.81 -> 0.92 mm
- net Net-(D166-DO): track 0.92 -> 3.55 mm
- net Net-(D165-DO): track 3.55 -> 0.92 mm
- net Net-(D83-DO): track 2.40 -> 0.00 mm
- net Earth: track 75.1 -> 77.3 mm
- net +5V: track 63.5 -> 65.3 mm
- net Net-(D69-DO): track 0.92 -> 2.62 mm
- net Net-(D68-DO): track 2.62 -> 0.92 mm
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
Commit message: [HW] Assign all parts
Parts:
- C6, C7: value 47pF -> 22pF
- J2, J3: value Interboard -> Interboard-F1
- J4: value Interboard -> Interboard-F2
- J5, J6: value Interboard -> Interboard-M1
- J7: value Interboard -> Interboard-M2
- R5, R6: value 27 -> 0
Connections:
- U3 pad 10: Earth -> unconnected-(U3-PIN10-Pad10)
- U3 pad 15: Earth -> unconnected-(U3-PIN15-Pad15)
- U3 pad 16: Earth -> unconnected-(U3-PIN16-Pad16)
Routing:
- net Earth: track 77.3 -> 75.7 mm, vias 21 -> 24

Commit message: [HW] Panelized and fab outputs generated
Parts:
- added mouse-bite-2mm-slot: VAL**, Panelization:mouse-bite-2mm-slot_round, F.Cu at (40.0, 40.0)
- added mouse-bite-2mm-slot: VAL**, Panelization:mouse-bite-2mm-slot_round, F.Cu at (40.0, 60.0)
- added mouse-bite-2mm-slot: VAL**, Panelization:mouse-bite-2mm-slot_round, F.Cu at (95.0, 60.0)
- added mouse-bite-2mm-slot: VAL**, Panelization:mouse-bite-2mm-slot_round, F.Cu at (60.0, 60.0)
- added mouse-bite-2mm-slot: VAL**, Panelization:mouse-bite-2mm-slot_round, F.Cu at (75.0, 40.0)
- added mouse-bite-2mm-slot: VAL**, Panelization:mouse-bite-2mm-slot_round, F.Cu at (75.0, 60.0)
- added mouse-bite-2mm-slot: VAL**, Panelization:mouse-bite-2mm-slot_round, F.Cu at (95.0, 40.0)
- added mouse-bite-2mm-slot: VAL**, Panelization:mouse-bite-2mm-slot_round, F.Cu at (60.0, 40.0)
- moved C1 5.00 mm to (88.5, 46.7)
- moved C10 5.00 mm to (82.0, 47.1)
- moved C11 5.00 mm to (81.5, 48.5)
- moved C12 5.00 mm to (85.2, 52.7)
- moved C13 5.00 mm to (76.2, 42.9)
- moved C14 5.00 mm to (78.1, 45.9)
- moved C15 5.00 mm to (82.3, 57.0)
- moved C16 5.00 mm to (87.7, 57.0)
- moved C2 5.00 mm to (89.5, 46.7)
- moved C3 5.00 mm to (91.0, 45.4)
- moved C4 5.00 mm to (92.3, 43.4)
- moved C5 5.00 mm to (74.3, 53.1)
- moved C6 5.00 mm to (79.1, 51.9)
- moved C7 5.00 mm to (79.1, 53.8)
- moved C8 5.00 mm to (82.3, 59.5)
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Other:
- board size 56.6 x 27.6 mm -> 72.9 x 38 mm

Commit message: [HW] Go through every part an ensure it matches the JLCPCB variant
Parts:
- J1: footprint Connector_USB:USB_C_Receptacle_GCT_USB4105-xx-A_16P_TopMnt_Horizontal -> EasyEDA2KiCad:USB-C-SMD_G-SWITCH_GT-USB-9010AB
- J2, J3: footprint Connector_PinSocket_1.27mm:PinSocket_2x02_P1.27mm_Vertical_SMD -> EasyEDA2KiCad:HDR-SMD_4P-P1.27-V-F-R2-C2-LS4.8
- J4: footprint Connector_PinSocket_1.27mm:PinSocket_2x04_P1.27mm_Vertical_SMD -> EasyEDA2KiCad:HDR-SMD_8P-P1.27-V-F-R2-C4-LS4.8
- J5, J6: footprint Connector_PinHeader_1.27mm:PinHeader_2x02_P1.27mm_Vertical_SMD -> EasyEDA2KiCad:HDR-SMD_4P-P1.27-V-M-R2-C2-S1.27-LS5.5
- U1: footprint MCU_Espressif_Official:ESP32-C3-MINI-1 -> EasyEDA2KiCad:WIFIM-SMD_ESP32-C3-MINI-1
- U3: footprint BNO055:LGA28R50P4X10_380X520X100 -> EasyEDA2KiCad:LGA-28_L5.2-W3.8-P0.50-BL
- moved U1 2.70 mm to (85.0, 50.0)
- moved J1 1.33 mm to (85.0, 59.4)
- turned J2 to 180 degrees
- turned J3 to 180 degrees
- turned J4 to 0 degrees
- turned J5 to 0 degrees
- turned J6 to 0 degrees
- turned U3 to -90 degrees

Commit message: [Hw] Fix component issues with JLCPCB Placement Still Need Fixes: U1: ESP32 (it's offset) U2: 3V3 Reg (Rotated) D1: USB Data ESD (Rotated, check that Footprint matches) D2: USB PWR ESD (Rotated?) J1: USB (Footprint generating DRC Errors) J7: 8P Interboard M (Missing LCSC Part, wait for it to be added)
Parts:
- D1: footprint TPD2EUSB30DRTR:DRT0003A -> EasyEDA2KiCad:SOT-723_L1.2-W0.8-P0.80-LS1.2-BR
- U2: footprint Package_TO_SOT_SMD:SOT-23-5 -> EasyEDA2KiCad:SOT-25-5_L2.9-W1.6-P0.95-LS2.8-BL
- U4: footprint Package_TO_SOT_SMD:SOT-363_SC-70-6 -> EasyEDA2KiCad:SC-70-6_L2.2-W1.3-P0.65-LS2.2-BR
- moved U1 2.49 mm to (85.0, 47.5), turned to 0 degrees
- turned U2 to 0 degrees
- turned U4 to 90 degrees

Commit message: Fixed a few placement correlation issues
Still TODO:
J1: USB (Footprint generating DRC Errors)
J7: Interboard (Missing LCSC Part, wait for it to be added)
Parts:
- moved U1 2.49 mm to (85.0, 50.0)
- turned D1 to 180 degrees
- turned D2 to 0 degrees
- turned U2 to 180 degrees
Routing:
- net Earth: track 75.7 -> 73.8 mm
