File: Small_Pendant/MCU.kicad_sch (KiCad schematic)
At the start: 41 parts, among them J1 USB_C_Receptacle_USB2.0_16P, Q1 MBT3904DW1T3G, SW1 SW_Push, SW2 SW_Push, SW3 SW_Push, U1 CP2102N-Axx-xQFN24, U2 SN74LVC1T45DCK, U3 ESP32-C3-MINI-1, U4 BNO055

Commit message: [HW] Added ESD Diode, Added VREG TODO: Connectors TODO?: Status LEDs (PWR vs Boot) (LED built in is a good idea to have, could blink every second to show alive-ness)
Parts:
- added C14: 10uF, Capacitor_SMD:C_0402_1005Metric, symbol Device:C
- added D1: TPD2EUSB30, TPD2EUSB30DRTR:DRT0003A, symbol TPD2EUSB30DRTR:TPD2EUSB30
- added R16: 100k, Resistor_SMD:R_0402_1005Metric, symbol Device:R_US
- added U5: AP2112K-3.3, Package_TO_SOT_SMD:SOT-23-5, symbol Regulator_Linear:AP2112K-3.3
Connections:
- net +3V3: now also C14.1, U5.5 (VOUT)
- net +5V: now also R16.1, U5.1 (VIN)
- net Earth: now also C14.2, D1.3 (GND), U5.2 (GND)
- net USB_D+: now also D1.1 (IO1)
- net USB_D-: now also D1.2 (IO2)
- new net: R16.2, U5.3 (EN)
Other:
- note added: "Colors"
- note added: "Patterns (And Wakeup)"
- moved on the sheet: C28, R12, R15

Commit message: [HW] More Rearrangement TODO: Renumber all components, so they're not dumb Also pick some goddamn LEDs so I can use D* and add that to renumbering
Parts:
- added C13: 10uF, Capacitor_SMD:C_0402_1005Metric, symbol Device:C
Connections:
- net +5V: now also C13.1
- net Earth: now also C13.2
Changed lines of the file:
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@@
 	)
 	(junction
+		(at 33.02 33.02)
+		(diameter 0)
+		(color 0 0 0 0)
+	)
+	(junction
 		(at 127 146.05)
 		(diameter 0)
@@
 	(wire
 		(pts
+			(xy 33.02 40.64) (xy 33.02 43.18)
+		)
+		(stroke
+			(width 0)
+			(type default)
+		)
+	)
+	(wire
+		(pts
 			(xy 63.5 40.64) (xy 63.5 43.18)
 		)
@@
 	(wire
 		(pts
+			(xy 33.02 43.18) (xy 53.34 43.18)
+		)
+		(stroke
+			(width 0)
+			(type default)
+		)
+	)
+	(wire
+		(pts
 			(xy 264.16 45.72) (xy 264.16 43.18)
 		)
@@
 					(unit 1)
 				)
+			)
+		)
+	)
+	(symbol
+		(lib_id "Device:C")
+		(at 33.02 36.83 0)
+		(mirror y)
+		(unit 1)
+		(exclude_from_sim no)
+		(in_bom yes)
+		(on_board yes)
+		(dnp no)
+		(property "Reference" "C13"
+			(at 29.21 35.5599 0)
+			(effects
+				(font
+					(size 1.27 1.27)
+				)
+				(justify left)
+			)
+		)
+		(property "Value" "10uF"
+			(at 29.21 38.0999 0)
+			(effects
+				(font
+					(size 1.27 1.27)
+				)
+				(justify left)
+			)
+		)
+		(property "Footprint" "Capacitor_SMD:C_0402_1005Metric"
+			(at 32.0548 40.64 0)
+			(effects
+				(font
+					(size 1.27 1.27)
+				)
+				(hide yes)
+			)
+		)
+		(property "Datasheet" "~"
+			(at 33.02 36.83 0)
+			(effects
+				(font
+					(size 1.27 1.27)
+				)
+				(hide yes)
+			)
+		)
+		(property "Description" "Unpolarized capacitor"
+			(at 33.02 36.83 0)
+			(effects
+				(font
+					(size 1.27 1.27)
+				)
+				(hide yes)
+			)
+		)
+		(property "MAXIMUM_PACKAGE_HEIGHT" ""
+			(at 33.02 36.83 0)
+			(effects
+				(font
+					(size 1.27 1.27)
+				)
+				(hide yes)
+			)
+		)
+		(property "PARTREV" ""
+			(at 33.02 36.83 0)
+			(effects
+				(font
+					(size 1.27 1.27)
+				)
+				(hide yes)
+			)
+		)
+		(property "Part#" ""
+			(at 33.02 36.83 0)
+			(effects
+				(font
+					(size 1.27 1.27)
+				)
+				(hide yes)
+			)
+		)
+		(property "STANDARD" ""
+			(at 33.02 36.83 0)
+			(effects
+				(font
+					(size 1.27 1.27)
+				)
+				(hide yes)
+			)
+		)
+		(property "Sim.Device" ""
+			(at 33.02 36.83 0)
+			(effects
+				(font
+					(size 1.27 1.27)
+				)
+				(hide yes)
+			)
+		)
+		(property "Sim.Pins" ""
+			(at 33.02 36.83 0)
+			(effects
+				(font
+					(size 1.27 1.27)
+				)
+				(hide yes)
+			)
+		)
+		(property "Sim.Type" ""
+			(at 33.02 36.83 0)
+			(effects
+				(font
+					(size 1.27 1.27)
+				)
+				(hide yes)
+			)
+		)
+		(pin "1"
+		)
+		(pin "2"
+		)
+		(instances
+			(project "Small_Pendant"
+				(path "/e1f67532-4244-48a0-a633-004c4e91cc2f/14f335fc-598f-404a-bfcd-3d46c6f23e92"
+					(reference "C13")
+					(unit 1)
+				)

Commit message: [HW] Re-annotate components, which absolutely wrecked everything, need to re-do the layout again
Parts:
- added D2: LED, symbol Device:LED
- added R4: ????, symbol Device:R_US
- renumbered C25 to C1, C21 to C10, C22 to C11, C28 to C12, C20 to C13, C29 to C14, C19 to C15, C17 to C16, C18 to C17, C23 to C19, C26 to C2, C24 to C20, C27 to C3, C31 to C4, C30 to C5, C13 to C6, C14 to C7, C15 to C8, C16 to C9, R6 to R1, R2 to R10, R3 to R11, R15 to R12, R12 to R13, R13 to R14, R14 to R15, R4 to R16, R5 to R17, R7 to R2, R8 to R3, R1 to R5, R11 to R6, R16 to R7, R10 to R8, U3 to U1, U5 to U2, U1 to U3, U2 to U5
Connections:
- net Earth: now also D2.1 (K)
- net IMU_INT: now also U1.16 (GPIO10); no longer U1.19 (GPIO5/ADC2_CH0)
- net USR_BTN: now also U1.12 (GPIO0/ADC1_CH0/XTAL_32K_P); no longer U1.16 (GPIO10)
- net at U1.13 (GPIO1/ADC1_CH1/XTAL_32K_N): now also R4.1
- new net: D2.2 (A), R4.2
- no-connect marks 20 -> 18
Other:
- note removed: "TODO: Add Power Enable Pin for I2C Power (Maybe)"
- moved on the sheet: C3, C8, C9, R1

Commit message: [HW] Finished re-laying out the front
Parts:
- renumbered C19 to C18, C20 to C19, R2 to R1, R13 to R12, R12 to R13, R3 to R2, R1 to R3
Connections:
- net LED_DATA: now also U1.27 (GPIO19/USB_D+); no longer U1.22 (GPIO8)
- no-connect marks 18 -> 20
Other:
- moved on the sheet: C1, C2, C3, D2, R1, R2, R3, R4, U1

Commit message: [HW] Added Connectors, P1.27mm double wide headers
Parts:
- added J2: Conn_02x03_Counter_Clockwise, Connector_PinSocket_1.27mm:PinSocket_2x03_P1.27mm_Vertical_SMD, symbol Connector_Generic:Conn_02x03_Counter_Clockwise
- added J3: Conn_02x02_Counter_Clockwise, Connector_PinSocket_1.27mm:PinSocket_2x02_P1.27mm_Vertical_SMD, symbol Connector_Generic:Conn_02x02_Counter_Clockwise
Connections:
- net +5V: now also J2.1 (Pin_1), J2.2 (Pin_2), J3.1 (Pin_1), J3.2 (Pin_2)
- net Earth: now also J2.3 (Pin_3), J2.4 (Pin_4), J3.3 (Pin_3), J3.4 (Pin_4)
- net LED_DATA-5V: no longer names the net of U5.3 (A)
- net LED_DATA-5V: now also J2.5 (Pin_5), J2.6 (Pin_6)
Other:
- moved on the sheet: C16, C17

Commit message: Removed USB to UART IC, instead using the built in USB on the ESP32-C3 (JTAG/USB-CDC combo in hardware) Added another connector, so total of 5 of each power line (5A without melting?) Renumbered and cleaned up layout, now happy Also created simple test board (I guess, need to figure out how to install that)
Parts:
- removed C12: 1uf, Capacitor_SMD:C_0402_1005Metric, symbol Device:C
- removed C8: 100nF, Capacitor_SMD:C_0402_1005Metric, symbol Device:C
- removed C9: 10uF, Capacitor_SMD:C_0402_1005Metric, symbol Device:C
- removed J2: Conn_02x03_Counter_Clockwise, Connector_PinSocket_1.27mm:PinSocket_2x03_P1.27mm_Vertical_SMD, symbol Connector_Generic:Conn_02x03_Counter_Clockwise
- removed Q1: MBT3904DW1T3G, EasyEDA2KiCad:SOT-363-6_L2.2-W1.3-P0.65-LS2.1-BL, symbol EasyEDA2KiCad:MBT3904DW1T3G
- removed R12: 47k, Resistor_SMD:R_0402_1005Metric, symbol Device:R_US
- removed R13: 22k, Resistor_SMD:R_0402_1005Metric, symbol Device:R_US
- removed R5, R6, R9: 10k, Resistor_SMD:R_0402_1005Metric, symbol Device:R_US
- removed R8: 1k, Resistor_SMD:R_0402_1005Metric, symbol Device:R_US
- removed U3: CP2102N-Axx-xQFN24, Package_DFN_QFN:QFN-24-1EP_4x4mm_P0.5mm_EP2.6x2.6mm, symbol Interface_USB:CP2102N-Axx-xQFN24
- added J2, J4: Interboard, Connector_PinSocket_1.27mm:PinSocket_2x02_P1.27mm_Vertical_SMD, symbol Connector_Generic:Conn_02x02_Counter_Clockwise
- J3: value Conn_02x02_Counter_Clockwise -> Interboard
- renumbered C13 to C10, C14 to C11, C15 to C12, C16 to C13, C17 to C14, C18 to C15, C19 to C16, C10 to C6, C11 to C7, C6 to C8, C7 to C9, R16 to R10, R17 to R11, R10 to R5, R11 to R6, R14 to R8, R15 to R9, U4 to U3, U5 to U4
Connections:
- net +5V: now also J2.1 (Pin_1), J4.1 (Pin_1), J4.2 (Pin_2)
- net Earth: now also C6.1, C7.1, J2.2 (Pin_2), J4.3 (Pin_3), J4.4 (Pin_4); no longer C6.2, C7.2
- net LED_DATA: now also U1.22 (GPIO8); no longer U1.27 (GPIO19/USB_D+)
- net USB_D'+: now also C6.2, D1.2 (IO2), R5.1, U1.27 (GPIO19/USB_D+); no longer R6.2
- net USB_D'-: now also C7.2, D1.1 (IO1), R6.1, U1.26 (GPIO18/USB_D-); no longer R5.2
- net USB_D+: now also R5.2; no longer C7.1, D1.1 (IO1), R6.1
- net USB_D-: now also R6.2; no longer C6.1, D1.2 (IO2), R5.1
- net LED_BUILTIN: now reaches R4.1, U1.13 (GPIO1/ADC1_CH1/XTAL_32K_N)
- net at U4.3 (A): now also J2.3 (Pin_3), J2.4 (Pin_4)
- net EXT_RX: no longer names the net of U1.30 (GPIO20/U0RXD)
- net EXT_TX: no longer names the net of U1.31 (GPIO21/U0TXD)
- no-connect marks 20 -> 11
Other:
- note removed: "Autoprogram"
- note removed: "UART"
- moved on the sheet: C6, C7, D1, J3, R1, R2, R5, R6

Commit message: [HW] Add LED (green) That's all the parts, now need to spec caps and resistors
Parts:
- D1: footprint TPD2EUSB30DRTR:DRT0003A -> DRT0003A
- D2: value LED -> BLUE; footprint (none) -> LED_SMD:LED_0603_1608Metric; Part# (none) -> C965806
- R4: value ???? -> 1k3; footprint (none) -> Resistor_SMD:R_0402_1005Metric

Commit message: [HW] Add Test Points (need Footprints)
Parts:
- added TP1: TX, symbol Connector:TestPoint
- added TP2: RX, symbol Connector:TestPoint
- added TP3: 5V, symbol Connector:TestPoint
- added TP4: 3V3, symbol Connector:TestPoint
- added TP5: GND, symbol Connector:TestPoint
Connections:
- net +3V3: now also TP3.1
- net +5V: now also TP4.1
- net Earth: now also TP5.1
- net at U1.30 (GPIO20/U0RXD): now also TP2.1
- net at U1.31 (GPIO21/U0TXD): now also TP1.1
- no-connect marks 11 -> 9
Other:
- moved on the sheet: C6, C7
