File: Small_Pendant/MCU.kicad_sch (KiCad schematic)
At the start: 45 parts, among them J1 USB_C_Receptacle_USB2.0_16P, J2 Interboard, J3 Interboard, J4 Interboard, SW1 SW_Push, SW2 SW_Push, SW3 SW_Push, U1 ESP32-C3-MINI-1, U2 AP2112K-3.3, U3 BNO055, U4 SN74LVC1T45DCK

Commit message: [HW] Add Test Points [SW] Update the board configs correctly
Parts:
- D1: footprint DRT0003A -> TPD2EUSB30DRTR:DRT0003A
- TP1, TP2, TP5: footprint (none) -> TestPoint:TestPoint_Pad_0.5x0.5mm
- TP3: value 5V -> 3V3; footprint (none) -> TestPoint:TestPoint_Pad_0.5x0.5mm
- TP4: value 3V3 -> 5V; footprint (none) -> TestPoint:TestPoint_Pad_0.5x0.5mm
Changed lines of the file:
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@@
 	)
 	(junction
-		(at 76.2 158.75)
+		(at 67.31 105.41)
 		(diameter 0)
 		(color 0 0 0 0)
 	)
 	(junction
-		(at 240.03 74.93)
+		(at 76.2 158.75)
 		(diameter 0)
 		(color 0 0 0 0)
 	)
 	(junction
-		(at 203.2 73.66)
+		(at 240.03 74.93)
 		(diameter 0)
 		(color 0 0 0 0)
 	)
 	(junction
-		(at 67.31 105.41)
+		(at 203.2 73.66)
 		(diameter 0)
 		(color 0 0 0 0)
@@
 	)
 	(junction
-		(at 67.31 95.25)
-		(diameter 0)
-		(color 0 0 0 0)
-	)
-	(junction
 		(at 255.27 95.25)
 		(diameter 0)
@@
 	)
 	(junction
+		(at 67.31 95.25)
+		(diameter 0)
+		(color 0 0 0 0)
+	)
+	(junction
 		(at 200.66 58.42)
 		(diameter 0)
@@
 	(wire
 		(pts
+			(xy 67.31 95.25) (xy 67.31 105.41)
+		)
+		(stroke
+			(width 0)
+			(type default)
+		)
+	)
+	(wire
+		(pts
 			(xy 33.02 27.94) (xy 33.02 30.48)
 		)
@@
 	(wire
 		(pts
-			(xy 67.31 95.25) (xy 67.31 105.41)
-		)
-		(stroke
-			(width 0)
-			(type default)
-		)
-	)
-	(wire
-		(pts
 			(xy 67.31 105.41) (xy 67.31 107.95)
 		)
@@
 			)
 		)
-		(property "Footprint" ""
+		(property "Footprint" "TestPoint:TestPoint_Pad_0.5x0.5mm"
 			(at 195.58 31.75 0)
 			(effects
@@
 			)
 		)
-		(property "Footprint" ""
+		(property "Footprint" "TestPoint:TestPoint_Pad_0.5x0.5mm"
 			(at 182.88 31.75 0)
 			(effects
@@
 			)
 		)
-		(property "Value" "3V3"
+		(property "Value" "5V"
 			(at 148.59 125.222 0)
 			(effects
@@
 			)
 		)
-		(property "Footprint" ""
+		(property "Footprint" "TestPoint:TestPoint_Pad_0.5x0.5mm"
 			(at 143.51 130.81 0)
 			(effects
@@
 			)
 		)
-		(property "Footprint" ""
+		(property "Footprint" "TestPoint:TestPoint_Pad_0.5x0.5mm"
 			(at 148.59 130.81 0)
 			(effects
@@
 			)
 		)
-		(property "Value" "5V"
+		(property "Value" "3V3"
 			(at 143.51 125.222 0)
 			(effects
@@
 			)
 		)
-		(property "Footprint" ""
+		(property "Footprint" "TestPoint:TestPoint_Pad_0.5x0.5mm"
 			(at 138.43 130.81 0)
 			(effects
@@
 			)
 		)
-		(property "Footprint" "DRT0003A"
+		(property "Footprint" "TPD2EUSB30DRTR:DRT0003A"
 			(at 212.09 40.64 0)
 			(effects

Commit message: [HW] switched J4/7 to 2x4 connectors for more current capacity
Parts:
- removed J4: Interboard, Connector_PinSocket_1.27mm:PinSocket_2x02_P1.27mm_Vertical_SMD, symbol Connector_Generic:Conn_02x02_Counter_Clockwise
- added J4: Interboard, Connector_PinSocket_1.27mm:PinSocket_2x04_P1.27mm_Vertical_SMD, symbol Connector_Generic:Conn_02x04_Odd_Even
- D1: LCSC Part (none) -> C5182099; Part# C5182099 -> (none)
- D2: value BLUE -> GREEN; LCSC Part (none) -> C965806; Part# C965806 -> (none)
- J1: LCSC Part (none) -> C3020560; Part# C3020560 -> (none)
- SW1, SW2, SW3: LCSC Part (none) -> C18078117; Part# C18078117 -> (none)
- U1: LCSC Part (none) -> C2934569; Part# C2934569 -> (none)
- U2: LCSC Part (none) -> C51118; Part# C51118 -> (none)
- U3: LCSC Part (none) -> C93216; Part# C93216 -> (none)
- U4: LCSC Part (none) -> C9382; Part# C9382 -> (none)
Connections:
- net +5V: now also J4.1 (Pin_1), J4.2 (Pin_2), J4.3 (Pin_3), J4.4 (Pin_4)
- net Earth: now also J4.5 (Pin_5), J4.6 (Pin_6), J4.7 (Pin_7), J4.8 (Pin_8)

Commit message: [HW] Schematic and Layout/Routing Clean Up
Connections:
- net LED_BUILTIN: now also R4.2; no longer R4.1
- net at D2.2 (A): now also R4.1; no longer R4.2
- net LED_DATA_5V: now reaches J2.3 (Pin_3), J2.4 (Pin_4), U4.3 (A)
Other:
- note added: "Buttons"
- note added: "Color Cycle"
- note added: "Data Translation"
- note added: "Interboard"
- note added: "Power Test Points"
- note removed: "Colors"
- note removed: "Level Shift"
- moved on the sheet: C1, C10, C11, C12, C13, C14, C15, C16, C2, C3, C4, C5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

Commit message: [Docs] Lots added to the Readme, BOM, schematics,...
Parts:
- J1: LCSC Part C3020560 -> C2988366
Changed lines of the file:
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@@
 			)
 		)
-		(property "LCSC Part" "C3020560"
+		(property "LCSC Part" "C2988366"
 			(at 29.21 40.64 0)
 			(effects

Commit message: [HW] Clean up ESD Diode
Connections:
- net USB_D'+: no longer D1.2 (IO2)
- net USB_D'-: no longer D1.1 (IO1)
- net USB_D+: now also D1.1 (IO1)
- net USB_D-: now also D1.2 (IO2)
Other:
- moved on the sheet: C6, C7, D1, R5, R6

Commit message: [HW] Add Series Resistor and power ESD diode
Parts:
- added D2: ESD441DPLR, EasyEDA2KiCad:X2SON-2_L0.6-W0.3-P0.35_ESD441DPLR, symbol EasyEDA2KiCad:ESD441DPLR
- renumbered D2 to D3
Connections:
- net +5V: now also D2.1 (K)
- net Earth: now also D2.2 (A)
Other:
- moved on the sheet: C15, C16, R11

Commit message: [HW] Assign all parts
Parts:
- C1, C16, C8, C9: LCSC Part (none) -> C7472949
- C10, C13, C14, C2, C4, C5: LCSC Part (none) -> C1525
- C11: LCSC Part (none) -> C7393864
- C12, C15, C3: LCSC Part (none) -> C14445
- C6, C7: value 47pF -> 22pF; LCSC Part (none) -> C106203
- J2, J3: value Interboard -> Interboard-F1; LCSC Part (none) -> C5160799
- J4: value Interboard -> Interboard-F2; LCSC Part (none) -> C5160800
- R1, R2: LCSC Part (none) -> C25890
- R10, R11: LCSC Part (none) -> C25905
- R3, R8, R9: LCSC Part (none) -> C25744
- R4: LCSC Part (none) -> C25866
- R5, R6: value 27 -> 0; LCSC Part (none) -> C17168
- R7: LCSC Part (none) -> C25741
- TP1, TP2, TP3, TP4, TP5: now not fitted
Connections:
- net Earth: no longer U3.10 (PIN10), U3.15 (PIN15), U3.16 (PIN16)
- no-connect marks 9 -> 12

Commit message: [HW] Go through every part an ensure it matches the JLCPCB variant
Parts:
- J1: footprint Connector_USB:USB_C_Receptacle_GCT_USB4105-xx-A_16P_TopMnt_Horizontal -> EasyEDA2KiCad:USB-C-SMD_G-SWITCH_GT-USB-9010AB
- J2, J3: footprint Connector_PinSocket_1.27mm:PinSocket_2x02_P1.27mm_Vertical_SMD -> EasyEDA2KiCad:HDR-SMD_4P-P1.27-V-F-R2-C2-LS4.8
- J4: footprint Connector_PinSocket_1.27mm:PinSocket_2x04_P1.27mm_Vertical_SMD -> EasyEDA2KiCad:HDR-SMD_8P-P1.27-V-F-R2-C4-LS4.8; LCSC Part C5160800 -> C5160801
- U1: footprint MCU_Espressif_Official:ESP32-C3-MINI-1 -> EasyEDA2KiCad:WIFIM-SMD_ESP32-C3-MINI-1
- U3: footprint BNO055:LGA28R50P4X10_380X520X100 -> EasyEDA2KiCad:LGA-28_L5.2-W3.8-P0.50-BL
Connections:
- net at J1.S1 (SHIELD): now also J1.S2 (SHIELD), J1.S3 (SHIELD), J1.S4 (SHIELD)
Changed lines of the file:
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@@
 			)
 		)
-		(property "Footprint" "Connector_PinSocket_1.27mm:PinSocket_2x02_P1.27mm_Vertical_SMD"
+		(property "Footprint" "EasyEDA2KiCad:HDR-SMD_4P-P1.27-V-F-R2-C2-LS4.8"
 			(at 81.28 134.62 0)
 			(effects
@@
 			)
 		)
-		(property "Footprint" "Connector_USB:USB_C_Receptacle_GCT_USB4105-xx-A_16P_TopMnt_Horizontal"
+		(property "Footprint" "EasyEDA2KiCad:USB-C-SMD_G-SWITCH_GT-USB-9010AB"
 			(at 33.02 40.64 0)
 			(effects
@@
 		(pin "A1"
 		)
+		(pin "S2"
+		)
+		(pin "S3"
+		)
+		(pin "S4"
+		)
 		(instances
 			(project "Small_Pendant"
@@
 			)
 		)
-		(property "Footprint" "BNO055:LGA28R50P4X10_380X520X100"
+		(property "Footprint" "EasyEDA2KiCad:LGA-28_L5.2-W3.8-P0.50-BL"
 			(at 156.21 139.7 0)
 			(effects
@@
 			)
 		)
-		(property "Footprint" "Connector_PinSocket_1.27mm:PinSocket_2x02_P1.27mm_Vertical_SMD"
+		(property "Footprint" "EasyEDA2KiCad:HDR-SMD_4P-P1.27-V-F-R2-C2-LS4.8"
 			(at 81.28 147.32 0)
 			(effects
@@
 			)
 		)
-		(property "Footprint" "MCU_Espressif_Official:ESP32-C3-MINI-1"
+		(property "Footprint" "EasyEDA2KiCad:WIFIM-SMD_ESP32-C3-MINI-1"
 			(at 181.61 95.25 0)
 			(effects
@@
 			)
 		)
-		(property "Footprint" "Connector_PinSocket_1.27mm:PinSocket_2x04_P1.27mm_Vertical_SMD"
+		(property "Footprint" "EasyEDA2KiCad:HDR-SMD_8P-P1.27-V-F-R2-C4-LS4.8"
 			(at 81.28 160.02 0)
 			(effects
@@
 			)
 		)
-		(property "Datasheet" "https://www.lcsc.com/datasheet/lcsc_datasheet_2411201843_DEALON-DW127S-22-06-43_C5160800.pdf"
+		(property "Datasheet" "https://www.lcsc.com/datasheet/lcsc_datasheet_2411201842_DEALON-DW127S-22-08-43_C5160801.pdf"
 			(at 81.28 160.02 0)
 			(effects
@@
 			)
 		)
-		(property "LCSC Part" "C5160800"
+		(property "LCSC Part" "C5160801"
 			(at 81.28 160.02 0)
 			(effects
