File: Small_Pendant/LED-Support.kicad_sch (KiCad schematic)
At the start: 15 parts, among them J5 Interboard, J6 Interboard, J7 Interboard

Commit message: [HW] Add Series Resistor and power ESD diode
Parts:
- added R12: 470, Resistor_SMD:R_0402_1005Metric, symbol Device:R_US
Connections:
- net DATA_IN: now also R12.2; no longer J5.3 (Pin_3), J5.4 (Pin_4)
- new net: J5.3 (Pin_3), J5.4 (Pin_4), R12.1
Changed lines of the file:
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@@
+	(wire
+		(pts
+			(xy 50.8 68.58) (xy 53.34 68.58)
+		)
+		(stroke
+			(width 0)
+			(type default)
+		)
+	)
 	(wire
 		(pts
@@
 	(global_label "DATA_IN"
 		(shape output)
-		(at 43.18 68.58 0)
+		(at 53.34 68.58 0)
 		(fields_autoplaced yes)
 		(effects
@@
 		)
 		(property "Intersheetrefs" "${INTERSHEET_REFS}"
-			(at 53.4829 68.58 0)
+			(at 63.6429 68.58 0)
 			(effects
 				(font
@@
 			)
 		)
+	)
+	(symbol
+		(lib_id "Device:R_US")
+		(at 46.99 68.58 90)
+		(unit 1)
+		(exclude_from_sim no)
+		(in_bom yes)
+		(on_board yes)
+		(dnp no)
+		(property "Reference" "R12"
+			(at 46.99 64.008 90)
+			(effects
+				(font
+					(size 1.27 1.27)
+				)
+			)
+		)
+		(property "Value" "470"
+			(at 46.99 66.04 90)
+			(effects
+				(font
+					(size 1.27 1.27)
+				)
+			)
+		)
+		(property "Footprint" "Resistor_SMD:R_0402_1005Metric"
+			(at 47.244 67.564 90)
+			(effects
+				(font
+					(size 1.27 1.27)
+				)
+				(hide yes)
+			)
+		)
+		(property "Datasheet" "~"
+			(at 46.99 68.58 0)
+			(effects
+				(font
+					(size 1.27 1.27)
+				)
+				(hide yes)
+			)
+		)
+		(property "Description" "Resistor, US symbol"
+			(at 46.99 68.58 0)
+			(effects
+				(font
+					(size 1.27 1.27)
+				)
+				(hide yes)
+			)
+		)
+		(property "MAXIMUM_PACKAGE_HEIGHT" ""
+			(at 46.99 68.58 0)
+			(effects
+				(font
+					(size 1.27 1.27)
+				)
+				(hide yes)
+			)
+		)
+		(property "PARTREV" ""
+			(at 46.99 68.58 0)
+			(effects
+				(font
+					(size 1.27 1.27)
+				)
+				(hide yes)
+			)
+		)
+		(property "STANDARD" ""
+			(at 46.99 68.58 0)
+			(effects
+				(font
+					(size 1.27 1.27)
+				)
+				(hide yes)
+			)
+		)
+		(property "Sim.Device" ""
+			(at 46.99 68.58 0)
+			(effects
+				(font
+					(size 1.27 1.27)
+				)
+				(hide yes)
+			)
+		)
+		(property "Sim.Pins" ""
+			(at 46.99 68.58 0)
+			(effects
+				(font
+					(size 1.27 1.27)
+				)
+				(hide yes)
+			)
+		)
+		(property "Sim.Type" ""
+			(at 46.99 68.58 0)
+			(effects
+				(font
+					(size 1.27 1.27)
+				)
+				(hide yes)
+			)
+		)
+		(property "LCSC Part" ""
+			(at 46.99 68.58 0)
+			(effects
+				(font
+					(size 1.27 1.27)
+				)
+				(hide yes)
+			)
+		)
+		(pin "2"
+		)
+		(pin "1"
+		)
+		(instances
+			(project "Small_Pendant"
+				(path "/e1f67532-4244-48a0-a633-004c4e91cc2f/0aa044a8-3060-48ad-928a-e0b7e1b97858"
+					(reference "R12")
+					(unit 1)
+				)
+			)
+		)

Commit message: [HW] Assign all parts
Parts:
- C17, C18, C19, C20, C21, C22, C23, C24, C25, C26, C27, C28: LCSC Part (none) -> C1525
- J5, J6: value Interboard -> Interboard-M1; LCSC Part (none) -> C5160758
- J7: value Interboard -> Interboard-M2; LCSC Part (none) -> C5160759
- R12: LCSC Part (none) -> C25117
Changed lines of the file:
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@@
 			)
 		)
-		(property "Datasheet" "~"
+		(property "Datasheet" "https://www.lcsc.com/datasheet/lcsc_datasheet_2411221126_UNI-ROYAL-Uniroyal-Elec-0402WGF4700TCE_C25117.pdf"
 			(at 46.99 68.58 0)
 			(effects
@@
 			)
 		)
-		(property "LCSC Part" ""
+		(property "LCSC Part" "C25117"
 			(at 46.99 68.58 0)
 			(effects
@@
 			)
 		)
-		(property "Datasheet" "~"
+		(property "Datasheet" "https://www.lcsc.com/datasheet/lcsc_datasheet_2304140030_Samsung-Electro-Mechanics-CL05B104KO5NNNC_C1525.pdf"
 			(at 162.56 33.02 0)
 			(effects
@@
 			)
 		)
-		(property "LCSC Part" ""
+		(property "LCSC Part" "C1525"
 			(at 162.56 33.02 0)
 			(effects
@@
 			)
 		)
-		(property "Value" "Interboard"
+		(property "Value" "Interboard-M1"
 			(at 31.75 77.47 0)
 			(effects
@@
 			)
 		)
-		(property "Datasheet" "~"
+		(property "Datasheet" "https://www.lcsc.com/datasheet/lcsc_datasheet_2411201840_DEALON-DZ127S-22-04-55_C5160758.pdf"
 			(at 30.48 81.28 0)
 			(effects
@@
 			)
 		)
-		(property "LCSC Part" ""
+		(property "LCSC Part" "C5160758"
 			(at 30.48 81.28 0)
 			(effects
@@
 			)
 		)
-		(property "Value" "Interboard"
+		(property "Value" "Interboard-M2"
 			(at 31.75 106.172 90)
 			(effects
@@
 			)
 		)
-		(property "Datasheet" "~"
+		(property "Datasheet" "https://www.lcsc.com/datasheet/lcsc_datasheet_2411201840_DEALON-DZ127S-22-06-55_C5160759.pdf"
 			(at 30.48 93.98 0)
 			(effects
@@
 		)
 		(property "Description" "Generic connector, double row, 02x04, odd/even pin numbering scheme (row 1 odd numbers, row 2 even numbers), script generated (kicad-library-utils/schlib/autogen/connector/)"
+			(at 30.48 93.98 0)
+			(effects
+				(font
+					(size 1.27 1.27)
+				)
+				(hide yes)
+			)
+		)
+		(property "LCSC Part" "C5160759"
 			(at 30.48 93.98 0)
 			(effects
@@
 			)
 		)
-		(property "Datasheet" "~"
+		(property "Datasheet" "https://www.lcsc.com/datasheet/lcsc_datasheet_2304140030_Samsung-Electro-Mechanics-CL05B104KO5NNNC_C1525.pdf"
 			(at 148.59 33.02 0)
 			(effects
@@
 			)
 		)
-		(property "LCSC Part" ""
+		(property "LCSC Part" "C1525"
 			(at 148.59 33.02 0)
 			(effects
@@
 			)
 		)
-		(property "Datasheet" "~"
+		(property "Datasheet" "https://www.lcsc.com/datasheet/lcsc_datasheet_2304140030_Samsung-Electro-Mechanics-CL05B104KO5NNNC_C1525.pdf"
 			(at 22.86 33.02 0)
 			(effects
@@
 			)
 		)
-		(property "LCSC Part" ""
+		(property "LCSC Part" "C1525"
 			(at 22.86 33.02 0)
 			(effects
@@
 			)
 		)
-		(property "Datasheet" "~"
+		(property "Datasheet" "https://www.lcsc.com/datasheet/lcsc_datasheet_2304140030_Samsung-Electro-Mechanics-CL05B104KO5NNNC_C1525.pdf"
 			(at 92.71 33.02 0)
 			(effects
@@
 			)
 		)
-		(property "LCSC Part" ""
+		(property "LCSC Part" "C1525"
 			(at 92.71 33.02 0)
 			(effects
@@
 			)
 		)
-		(property "Datasheet" "~"
+		(property "Datasheet" "https://www.lcsc.com/datasheet/lcsc_datasheet_2304140030_Samsung-Electro-Mechanics-CL05B104KO5NNNC_C1525.pdf"
 			(at 78.74 33.02 0)
 			(effects
@@
 			)
 		)
-		(property "LCSC Part" ""
+		(property "LCSC Part" "C1525"
 			(at 78.74 33.02 0)
 			(effects
@@
 			)
 		)
-		(property "Datasheet" "~"
+		(property "Datasheet" "https://www.lcsc.com/datasheet/lcsc_datasheet_2304140030_Samsung-Electro-Mechanics-CL05B104KO5NNNC_C1525.pdf"
 			(at 36.83 33.02 0)
 			(effects
@@
 			)
 		)
-		(property "LCSC Part" ""
+		(property "LCSC Part" "C1525"
 			(at 36.83 33.02 0)
 			(effects
@@
 			)
 		)
-		(property "Datasheet" "~"
+		(property "Datasheet" "https://www.lcsc.com/datasheet/lcsc_datasheet_2304140030_Samsung-Electro-Mechanics-CL05B104KO5NNNC_C1525.pdf"
 			(at 176.53 33.02 0)
 			(effects
@@
 			)
 		)
-		(property "LCSC Part" ""
+		(property "LCSC Part" "C1525"
 			(at 176.53 33.02 0)
 			(effects
@@
 			)
 		)
-		(property "Value" "Interboard"
+		(property "Value" "Interboard-M1"
 			(at 31.75 64.77 0)
 			(effects
@@
 			)
 		)
-		(property "Datasheet" "~"
+		(property "Datasheet" "https://www.lcsc.com/datasheet/lcsc_datasheet_2411201840_DEALON-DZ127S-22-04-55_C5160758.pdf"
 			(at 30.48 68.58 0)
 			(effects
@@
 			)
 		)
-		(property "LCSC Part" ""
+		(property "LCSC Part" "C5160758"
 			(at 30.48 68.58 0)
 			(effects
@@
 			)
 		)
-		(property "Datasheet" "~"
+		(property "Datasheet" "https://www.lcsc.com/datasheet/lcsc_datasheet_2304140030_Samsung-Electro-Mechanics-CL05B104KO5NNNC_C1525.pdf"
 			(at 50.8 33.02 0)
 			(effects
@@
 			)
 		)
-		(property "LCSC Part" ""
+		(property "LCSC Part" "C1525"
 			(at 50.8 33.02 0)
 			(effects
@@
 			)
 		)
-		(property "Datasheet" "~"
+		(property "Datasheet" "https://www.lcsc.com/datasheet/lcsc_datasheet_2304140030_Samsung-Electro-Mechanics-CL05B104KO5NNNC_C1525.pdf"
 			(at 134.62 33.02 0)
 			(effects
@@
 			)
 		)
-		(property "LCSC Part" ""
+		(property "LCSC Part" "C1525"
 			(at 134.62 33.02 0)
 			(effects
@@
 			)
 		)
-		(property "Datasheet" "~"
+		(property "Datasheet" "https://www.lcsc.com/datasheet/lcsc_datasheet_2304140030_Samsung-Electro-Mechanics-CL05B104KO5NNNC_C1525.pdf"
 			(at 120.65 33.02 0)
 			(effects
@@
 			)
 		)
-		(property "LCSC Part" ""
+		(property "LCSC Part" "C1525"
 			(at 120.65 33.02 0)
 			(effects
@@
 			)
 		)
-		(property "Datasheet" "~"
+		(property "Datasheet" "https://www.lcsc.com/datasheet/lcsc_datasheet_2304140030_Samsung-Electro-Mechanics-CL05B104KO5NNNC_C1525.pdf"
 			(at 64.77 33.02 0)
 			(effects
@@
 			)
 		)
-		(property "LCSC Part" ""
+		(property "LCSC Part" "C1525"
 			(at 64.77 33.02 0)
 			(effects
@@
 			)
 		)
-		(property "Datasheet" "~"
+		(property "Datasheet" "https://www.lcsc.com/datasheet/lcsc_datasheet_2304140030_Samsung-Electro-Mechanics-CL05B104KO5NNNC_C1525.pdf"
 			(at 106.68 33.02 0)
 			(effects
@@
 			)
 		)
-		(property "LCSC Part" ""
+		(property "LCSC Part" "C1525"
 			(at 106.68 33.02 0)
 			(effects

Commit message: [HW] Go through every part an ensure it matches the JLCPCB variant
Parts:
- J5, J6: footprint Connector_PinHeader_1.27mm:PinHeader_2x02_P1.27mm_Vertical_SMD -> EasyEDA2KiCad:HDR-SMD_4P-P1.27-V-M-R2-C2-S1.27-LS5.5
- J7: LCSC Part C5160759 -> C5160760
Changed lines of the file:
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@@
 			)
 		)
-		(property "Footprint" "Connector_PinHeader_1.27mm:PinHeader_2x02_P1.27mm_Vertical_SMD"
+		(property "Footprint" "EasyEDA2KiCad:HDR-SMD_4P-P1.27-V-M-R2-C2-S1.27-LS5.5"
 			(at 30.48 81.28 0)
 			(effects
@@
 			)
 		)
-		(property "Datasheet" "https://www.lcsc.com/datasheet/lcsc_datasheet_2411201840_DEALON-DZ127S-22-06-55_C5160759.pdf"
+		(property "Datasheet" "https://www.lcsc.com/datasheet/lcsc_datasheet_2411201840_DEALON-DZ127S-22-08-55_C5160760.pdf"
 			(at 30.48 93.98 0)
 			(effects
@@
 			)
 		)
-		(property "LCSC Part" "C5160759"
+		(property "LCSC Part" "C5160760"
 			(at 30.48 93.98 0)
 			(effects
@@
 			)
 		)
-		(property "Footprint" "Connector_PinHeader_1.27mm:PinHeader_2x02_P1.27mm_Vertical_SMD"
+		(property "Footprint" "EasyEDA2KiCad:HDR-SMD_4P-P1.27-V-M-R2-C2-S1.27-LS5.5"
 			(at 30.48 68.58 0)
 			(effects

Commit message: [HW] Fix 'all' component issue, still unsure of the male 8pin jumper
Parts:
- J7: footprint Connector_PinHeader_1.27mm:PinHeader_2x04_P1.27mm_Vertical_SMD -> EasyEDA2KiCad:HDR-SMD_8P-P1.27-V-M-R2-C4-S1.27-LS5.5_Guess
Changed lines of the file:
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@@
 			)
 		)
-		(property "Footprint" "Connector_PinHeader_1.27mm:PinHeader_2x04_P1.27mm_Vertical_SMD"
+		(property "Footprint" "EasyEDA2KiCad:HDR-SMD_8P-P1.27-V-M-R2-C4-S1.27-LS5.5_Guess"
 			(at 30.48 93.98 0)
 			(effects

Commit message: [HW] Finalize production outputs for fab Not 100% sure everything is fine, but it should be
Parts:
- J7: footprint EasyEDA2KiCad:HDR-SMD_8P-P1.27-V-M-R2-C4-S1.27-LS5.5_Guess -> EasyEDA2KiCad:HDR-SMD_8P-P1.27-V-M-R2-C4-W5.5
Changed lines of the file:
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@@
 			)
 		)
-		(property "Footprint" "EasyEDA2KiCad:HDR-SMD_8P-P1.27-V-M-R2-C4-S1.27-LS5.5_Guess"
+		(property "Footprint" "EasyEDA2KiCad:HDR-SMD_8P-P1.27-V-M-R2-C4-W5.5"
 			(at 30.48 93.98 0)
 			(effects

Commit message: [HW] Add Missing Bootstrap Pin
Parts:
- renumbered R12 to R13
Changed lines of the file:
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@@
 		(on_board yes)
 		(dnp no)
-		(property "Reference" "R12"
+		(property "Reference" "R13"
 			(at 46.99 64.008 90)
 			(effects
@@
 			(project "Small_Pendant"
 				(path "/e1f67532-4244-48a0-a633-004c4e91cc2f/0aa044a8-3060-48ad-928a-e0b7e1b97858"
-					(reference "R12")
+					(reference "R13")
 					(unit 1)
 				)
